Commit message: [rolling][WIP] update urdf for horizontal model

File: robots/rolling/urdf/rolling_link.urdf.xacro (robot description, xacro)
@@ -6,5 +6,5 @@
     <link name="root">
       <inertial>
-        <origin xyz="0 0 0" rpy="0 0 0"/>
+        <origin xyz="0 0 1.2" rpy="0 0 0"/>
         <mass value="0.00001"/>
         <inertia
@@ -30,5 +30,5 @@
       </inertial>
       <visual>
-        <origin xyz="0 0 0" rpy="${pi / 2} 0 0" />
+        <origin xyz="0 0 0" rpy="0 0 0" />
         <geometry>
           <cylinder radius="${cylinder_radius}" length="0.1"/>
@@ -39,7 +39,7 @@
       </visual>
       <collision>
-        <origin xyz="0 0 0" rpy="${pi / 2} 0 0"/>
+        <origin xyz="0 0 0" rpy="0 0 0"/>
         <geometry>
-          <cylinder radius="${cylinder_radius}" length="0.3"/>
+          <cylinder radius="${cylinder_radius}" length="0.1"/>
         </geometry>
       </collision>
@@ -66,13 +66,13 @@
       <parent link="base_link"/>
       <child link="gimbal_link${child1}"/>
-      <origin rpy="0 ${pi/2} 0" xyz="${cylinder_radius} 0 0"/>
-      <axis xyz="1 0 0"/>
-      <dynamics damping="0.8" friction="0.0"/>
-    </joint>
-  <joint name="gimbal${child2}" type="revolute">
+      <origin rpy="0 0 0" xyz="${cylinder_radius} 0 0"/>
+      <axis xyz="1 0 0"/>
+      <dynamics damping="0.8" friction="0.0"/>
+    </joint>
+    <joint name="gimbal${child2}" type="revolute">
       <limit effort="6.6" lower="-1.57" upper="1.57" velocity="3.0"/>
       <parent link="base_link"/>
       <child link="gimbal_link${child2}"/>
-      <origin rpy="0 0 0" xyz="0 0 ${cylinder_radius}"/>
+      <origin rpy="0 0 0" xyz="0 -${cylinder_radius} 0"/>
       <axis xyz="1 0 0"/>
       <dynamics damping="0.8" friction="0.0"/>
@@ -82,5 +82,5 @@
       <parent link="base_link"/>
       <child link="gimbal_link${child3}"/>
-      <origin rpy="0 ${-pi/2} 0" xyz="${- cylinder_radius} 0 0"/>
+      <origin rpy="0 0 0" xyz="${- cylinder_radius} 0 0"/>
       <axis xyz="1 0 0"/>
       <dynamics damping="0.8" friction="0.0"/>
@@ -90,5 +90,5 @@
       <parent link="base_link"/>
       <child link="gimbal_link${child4}"/>
-      <origin rpy="0 ${pi} 0" xyz="0 0 ${- cylinder_radius}"/>
+      <origin rpy="0 0 0" xyz="0 ${cylinder_radius} 0"/>
       <axis xyz="1 0 0"/>
       <dynamics damping="0.8" friction="0.0"/>
@@ -140,5 +140,5 @@
       <inertial>
         <origin xyz="0 0 0" rpy="0 0 0"/>
-        <mass value="0.00001"/>
+        <mass value="0.2"/>
         <inertia
             ixx="0.000001" ixy="0.0" ixz="0.0"
