Commit message: [dragon] modify yaw joint range for 3link model

File: robots/dragon/urdf/dragon_link.urdf.xacro (robot description, xacro)
@@ -227,5 +227,5 @@
       </link>
       <joint name="joint${self}_yaw" type="revolute">
-        <limit effort="10.0" lower="${-pi/2}" upper="${pi/2}" velocity="0.1"/>
+        <limit effort="10.0" lower="${-pi}" upper="${pi}" velocity="0.1"/>
         <parent link="inter_joint${self}"/>
         <child link="link${child}"/>
