Commit message: tmp

File: robots/delta/urdf/20240319_mesh/rolling_link.urdf.xacro (robot description, xacro)
@@ -36,5 +36,5 @@
     <xacro:unless value="${self == child}">
       <joint name="joint${self}" type="revolute" >
-        <limit effort="20.0" lower="${-pi}" upper="${pi}" velocity="0.1"/>
+        <limit effort="100.0" lower="${-pi}" upper="${pi}" velocity="0.1"/>
         <parent link="link${self}" />
         <child  link="link${child}" />

File: robots/delta/urdf/common.xacro (robot description, xacro)
@@ -15,6 +15,6 @@
   <xacro:macro name="large_friction" params="link">
     <gazebo reference="${link}">
-      <mu1>100</mu1>
-      <mu2>100</mu2>
+      <mu1>10</mu1>
+      <mu2>10</mu2>
     </gazebo>
   </xacro:macro>
