Commit message: [mini_quadrotor] changed rotor joint model from continuous to revolute

File: robots/mini_quadrotor/urdf/robot.urdf (robot description, URDF)
Before this commit: robot module_quadrotor, 9 links, 8 joints
Joints:
- joint rotor1: type continuous -> revolute
- joint rotor2: type continuous -> revolute
- joint rotor3: type continuous -> revolute
- joint rotor4: type continuous -> revolute

Commit message: [mini_quadrotor] changed rotor joint to fixed type

File: robots/mini_quadrotor/urdf/robot.urdf (robot description, URDF)
Before this commit: robot module_quadrotor, 9 links, 8 joints
Joints:
- joint rotor1: type revolute -> fixed
- joint rotor2: type revolute -> fixed
- joint rotor3: type revolute -> fixed
- joint rotor4: type revolute -> fixed
