Commit message: [mini_quadrotor] add comment to use livox

File: robots/mini_quadrotor/urdf/robot_with_t265.urdf.xacro (robot description, xacro)
@@ -148,4 +148,15 @@
     </inertial>
   </xacro:extra_module>
+  <!-- livox mid360 -->
+  <xacro:extra_module name = "lidar_imu" parent = "main_body" visible = "0" > <!-- should be IMU frame -->
+    <origin xyz="0 0 0.1" rpy="0 0 ${pi / 2}"/> <!-- TODO: the true pos -->
+    <inertial>
+      <mass value="0" />
+      <origin xyz="0 0 0" rpy="0 0 0"/>
+      <inertia
+          ixx="0.0" ixy="0.0" ixz="0.0"
+          iyy="0.0" iyz="0.0" izz="0.0"/>
+    </inertial>
+  </xacro:extra_module>
   <!-- battery -->
   <xacro:extra_module name = "battery" parent = "main_body" visible = "1" model_url = "package://mini_quadrotor/urdf/mesh/turnigy_3S_2200mAh.dae" >
