Commit message: <debug> add uuv plugin but not reflect buoyancy to robot main body and debug mode

File: robots/mini_quadrotor/urdf/robot.gazebo.xacro (robot description, xacro)
@@ -7,8 +7,38 @@
   <!-- gazebo plugin for default controller and sensors -->
   <xacro:include filename="$(find aerial_robot_simulation)/xacro/spinal.gazebo.xacro" />
-  <xacro:gazebo_spinal robot_name="$(arg robot_name)" />
+  <xacro:gazebo_spinal robot_name="$(arg robot_name)" gps_frame="fc" />
   <gazebo reference="main_body">
     <mu1>0.1</mu1>
     <mu2>0.1</mu2>
   </gazebo>
+  <gazebo>
+    <plugin name="uuv_plugin" filename="libuuv_underwater_object_ros_plugin.so">
+      <fluid_density>1000.0</fluid_density>
+      <flow_velocity_topic>/hydrodynamics/current_velocity</flow_velocity_topic>
+      <debug>1</debug>
+      <link name="main_body">
+        <neutrally_buoyant>0</neutrally_buoyant>
+        <volume>0.0</volume>
+        <box>
+          <width>0.28</width>
+          <length>0.28</length>
+          <height>0.072</height>
+        </box>
+        <center_of_buoyancy>0 0 0</center_of_buoyancy>
+        <hydrodynamic_model>
+          <type>fossen</type>
+          <added_mass>
+            0 0 0 0 0 0
+            0 0 0 0 0 0
+            0 0 0 0 0 0
+            0 0 0 0 0 0
+            0 0 0 0 0 0
+            0 0 0 0 0 0
+          </added_mass>
+          <linear_damping> -0.1 -0.1 -0.1 -0.01 -0.01 -0.01</linear_damping>
+          <quadratic_damping>-0.2 -0.2 -0.4 -0.02 -0.02 -0.02</quadratic_damping>
+        </hydrodynamic_model>
+      </link>
+    </plugin>
+  </gazebo>
 </robot>

Commit message: [mini_quadrotor] fix link name from main_body to base_link for uuv_simulator compatibility and do not lump with fixed root_joint to load base_link as link

File: robots/mini_quadrotor/urdf/robot.gazebo.xacro (robot description, xacro)
@@ -8,7 +8,10 @@
   <xacro:include filename="$(find aerial_robot_simulation)/xacro/spinal.gazebo.xacro" />
   <xacro:gazebo_spinal robot_name="$(arg robot_name)" gps_frame="fc" />
-  <gazebo reference="main_body">
+  <gazebo reference="base_link">
     <mu1>0.1</mu1>
     <mu2>0.1</mu2>
+  </gazebo>
+  <gazebo reference="root_joint">
+    <disableFixedJointLumping>true</disableFixedJointLumping>
   </gazebo>
   <gazebo>
@@ -17,5 +20,5 @@
       <flow_velocity_topic>/hydrodynamics/current_velocity</flow_velocity_topic>
       <debug>1</debug>
-      <link name="main_body">
+      <link name="base_link">
         <neutrally_buoyant>0</neutrally_buoyant>
         <volume>0.0</volume>

File: robots/mini_quadrotor/urdf/robot.urdf.xacro (robot description, xacro)
@@ -15,5 +15,5 @@
   <!-- friction -->
   <xacro:macro name="damping_factor" params="link">
-    <gazebo reference="main_body">
+    <gazebo reference="base_link">
       <dampingFactor>0.00</dampingFactor>
     </gazebo>
@@ -40,5 +40,5 @@
     <joint name="rotor${id}" type="continuous">
       <limit effort="100.0" lower="${min_force}" upper="${max_force}" velocity="0.5"/>
-      <parent link="main_body"/>
+      <parent link="base_link"/>
       <child link="thrust${id}"/>
       <origin rpy="0 0 0" xyz="${x} ${y} ${z}"/>
@@ -89,10 +89,10 @@
   <joint name="root_joint" type="fixed">
     <parent link="root"/>
-    <child link="main_body"/>
+    <child link="base_link"/>
     <origin rpy="0 0 0" xyz="0 0 0"/>
     <axis xyz="0 0 1"/>
   </joint>
-  <!-- main_body -->
-  <link name="main_body">
+  <!-- base_link -->
+  <link name="base_link">
     <inertial>
       <mass value = "0.860" />
@@ -117,5 +117,5 @@
   </link>
   <!-- spinal -->
-  <xacro:extra_module name = "fc" parent = "main_body" visible = "0" >
+  <xacro:extra_module name = "fc" parent = "base_link" visible = "0" >
     <origin xyz="-0.02 -0.005 0.03" rpy="0 0 0"/>
     <inertial>
@@ -127,5 +127,5 @@
     </inertial>
   </xacro:extra_module>
-  <xacro:extra_module name = "magnet" parent = "main_body" visible = "0" >
+  <xacro:extra_module name = "magnet" parent = "base_link" visible = "0" >
     <origin xyz="0 0 0" rpy="0 0 0"/>
     <inertial>
@@ -138,5 +138,5 @@
   </xacro:extra_module>
   <!-- livox mid360 -->
-  <xacro:extra_module name = "lidar_imu" parent = "main_body" visible = "0" > <!-- should be IMU frame -->
+  <xacro:extra_module name = "lidar_imu" parent = "base_link" visible = "0" > <!-- should be IMU frame -->
     <origin xyz="${0.011} ${0.02329} ${0.0425 + 0.047 - 0.04412}" rpy="0 0 0"/> <!-- TODO: the true pos -->
     <inertial>
@@ -149,5 +149,5 @@
   </xacro:extra_module>
   <!-- battery -->
-  <xacro:extra_module name = "battery" parent = "main_body" visible = "1" model_url = "package://mini_quadrotor/urdf/mesh/turnigy_3S_2200mAh.dae" >
+  <xacro:extra_module name = "battery" parent = "base_link" visible = "1" model_url = "package://mini_quadrotor/urdf/mesh/turnigy_3S_2200mAh.dae" >
     <origin xyz="0.0 0 -0.035" rpy="${pi/2} 0 0"/>
     <inertial>
