Commit message: [dragon] add variable to urdf to set rotor joint for gazebo(continuous) and pinocchio(fixed)

File: robots/dragon/robots/quad/euclid_201709.gazebo.xacro (robot description, xacro)
@@ -3,4 +3,5 @@
     xmlns:xacro="http://www.ros.org/wiki/xacro" name="dragon" >
   <xacro:arg name="robot_name" default="dragon" />
+  <xacro:arg name="rotor_fixed" default="false"/>
   <!-- robot urdf -->
   <xacro:include filename="$(find dragon)/robots/quad/euclid_201709.urdf.xacro" />

File: robots/dragon/robots/quad/euclid_201709.urdf.xacro (robot description, xacro)
@@ -2,10 +2,11 @@
 <robot
     xmlns:xacro="http://www.ros.org/wiki/xacro" name="dragon" >
+  <xacro:arg name="rotor_fixed" default="false"/>
   <!-- temporary -->
   <xacro:include filename="$(find dragon)/urdf/dragon_common.xacro" />
   <xacro:include filename="$(find dragon)/urdf/dragon_link.urdf.xacro" />
-  <xacro:dragon_module self="1" child="2" baselink="false" />
-  <xacro:dragon_module self="2" child="3" baselink="true" />
-  <xacro:dragon_module self="3" child="4" baselink="false" />
-  <xacro:dragon_module self="4" child="4" baselink="false" />
+  <xacro:dragon_module self="1" child="2" baselink="false" rotor_fixed="$(arg rotor_fixed)"/>
+  <xacro:dragon_module self="2" child="3" baselink="true"  rotor_fixed="$(arg rotor_fixed)"/>
+  <xacro:dragon_module self="3" child="4" baselink="false" rotor_fixed="$(arg rotor_fixed)"/>
+  <xacro:dragon_module self="4" child="4" baselink="false" rotor_fixed="$(arg rotor_fixed)"/>
 </robot>

File: robots/dragon/urdf/dragon_link.urdf.xacro (robot description, xacro)
@@ -3,5 +3,5 @@
     xmlns:xacro="http://www.ros.org/wiki/xacro" name="dragon_link" >
   <!-- D-H kai description(different from prof.nakamura) -->
-  <xacro:macro name="dragon_module" params="self child baselink">
+  <xacro:macro name="dragon_module" params="self child baselink rotor_fixed:=false">
     <!-- link -->
     <link name="link${self}">
@@ -148,11 +148,32 @@
     </link>
     <!-- rotor -->
-    <joint name="rotor${self}" type="fixed">
-      <!-- <limit effort="100.0" lower="${min_force}" upper="${max_force}" velocity="0.5"/> -->
-      <parent link="gimbal${self}_pitch_module"/>
-      <child link="thrust${self}"/>
-      <origin rpy="0 0 0" xyz="0 0 0"/>
-      <axis xyz="0 0 1"/>
-    </joint>
+    <xacro:if value="${rotor_fixed}">
+      <joint name="rotor${self}" type="fixed">
+        <parent link="gimbal${self}_pitch_module"/>
+        <child link="thrust${self}"/>
+        <origin rpy="0 0 0" xyz="0 0 0"/>
+        <axis xyz="0 0 1"/>
+      </joint>
+    </xacro:if>
+    <xacro:unless value="${rotor_fixed}">
+      <joint name="rotor${self}" type="continuous">
+        <limit effort="100.0" lower="${min_force}" upper="${max_force}" velocity="0.5"/>
+        <parent link="gimbal${self}_pitch_module"/>
+        <child link="thrust${self}"/>
+        <origin rpy="0 0 0" xyz="0 0 0"/>
+        <axis xyz="0 0 1"/>
+      </joint>
+      <transmission name="rotor${self}_tran">
+        <type>transmission_interface/SimpleTransmission</type>
+        <joint name="rotor${self}">
+          <hardwareInterface>RotorInterface</hardwareInterface>
+        </joint>
+        <actuator name="rotor${self}">
+          <hardwareInterface>RotorInterface</hardwareInterface>
+          <mechanicalReduction>1</mechanicalReduction>
+        </actuator>
+      </transmission>
+      <xacro:friction self ="${self}"/>
+    </xacro:unless>
     <link name="thrust${self}">
       <inertial>
@@ -324,15 +345,4 @@
       </actuator>
     </transmission>
-    <!-- <transmission name="rotor${self}_tran"> -->
-    <!--   <type>transmission_interface/SimpleTransmission</type> -->
-    <!--   <joint name="rotor${self}"> -->
-    <!--     <hardwareInterface>RotorInterface</hardwareInterface> -->
-    <!--   </joint> -->
-    <!--   <actuator name="rotor${self}"> -->
-    <!--     <hardwareInterface>RotorInterface</hardwareInterface> -->
-    <!--     <mechanicalReduction>1</mechanicalReduction> -->
-    <!--   </actuator> -->
-    <!--   </transmission> -->
-    <!-- <xacro:friction self ="${self}"/> -->
   </xacro:macro>
 </robot>
