Commit message: [dragon] update urdf. change spinal position and joint parameters

File: robots/dragon/robots/quad/euclid_201709.urdf.xacro (robot description, xacro)
@@ -10,3 +10,36 @@
   <xacro:dragon_module self="3" child="4" baselink="false" rotor_fixed="$(arg rotor_fixed)"/>
   <xacro:dragon_module self="4" child="4" baselink="false" rotor_fixed="$(arg rotor_fixed)"/>
+  <!-- set the fcu frame -->
+  <link name="fc">
+    <inertial>
+      <origin xyz="0 0 0" rpy="0 0 0"/>
+      <mass value="0.00001"/>
+      <inertia
+          ixx="0.000001" ixy="0.0" ixz="0.0"
+          iyy="0.000001" iyz="0.0"
+          izz="0.000002"/>
+    </inertial>
+  </link>
+  <joint name="fc_joint" type="fixed">
+    <child link="fc"/>
+    <parent link="link1"/>
+    <origin rpy="0 0 0" xyz="0.316 -0.004 0.043"/>
+    <axis xyz="0 0 1"/>
+  </joint>
+    <joint name="end_effector_joint" type="fixed">
+    <parent link="link4"/>
+    <child link="link4_tip"/>
+    <origin xyz="${link_length} 0 0" rpy="0 0 0"/>
+    <axis xyz="0 0 1"/>
+  </joint>
+  <link name="link4_tip">
+    <inertial>
+      <origin xyz="0 0 0" rpy="0 0 0"/>
+      <mass value="0.00001"/>
+      <inertia
+          ixx="0.000001" ixy="0.0" ixz="0.0"
+          iyy="0.000001" iyz="0.0"
+          izz="0.000002"/>
+    </inertial>
+  </link>
 </robot>

File: robots/dragon/urdf/dragon_common.xacro (robot description, xacro)
@@ -18,5 +18,5 @@
   <m_f_rate value="0" /> <!-- drug torque rate -->
   <xacro:property name="max_force" value="30" /> <!-- [N] -->
-  <xacro:property name="min_force" value="2" /> <!-- [N] -->
+  <xacro:property name="min_force" value="0" /> <!-- [N] -->
   <xacro:macro name="link_model" params="type">
     <!-- box collision geometry does not work well for FCL -->

File: robots/dragon/urdf/dragon_link.urdf.xacro (robot description, xacro)
@@ -223,10 +223,10 @@
     <xacro:unless value="${self == child}">
       <joint name="joint${self}_pitch" type="revolute">
-        <limit effort="10.0" lower="${-pi/2}" upper="${pi/2}" velocity="0.1"/>
+        <limit effort="20.0" lower="${-pi/2}" upper="${pi/2}" velocity="6"/>
         <parent link="link${self}"/>
         <child link="inter_joint${self}"/>
         <origin rpy="0 0 0" xyz="${link_length} 0 0"/>
         <axis xyz="0 1 0"/>
-        <dynamics damping="0.9" friction="0.05"/>
+        <dynamics damping="0.1" friction="0.0"/>
       </joint>
       <!-- inter joint -->
@@ -248,10 +248,10 @@
       </link>
       <joint name="joint${self}_yaw" type="revolute">
-        <limit effort="10.0" lower="${-pi/2}" upper="${pi/2}" velocity="0.1"/>
+        <limit effort="20.0" lower="${-pi/2}" upper="${pi/2}" velocity="6"/>
         <parent link="inter_joint${self}"/>
         <child link="link${child}"/>
         <origin rpy="0 0 0" xyz="${2 * inter_joint_x_offset} 0 0"/>
         <axis xyz="0 0 1"/>
-        <dynamics damping="0.9" friction="0.05"/>
+        <dynamics damping="0.1" friction="0.0"/>
       </joint>
       <gazebo reference="inter_joint${self}">
@@ -276,23 +276,4 @@
         <child link="link${self}"/>
         <origin rpy="0 0 0" xyz="0 0 0"/>
-        <axis xyz="0 0 1"/>
-      </joint>
-    </xacro:if>
-    <!-- set the fcu frame -->
-    <xacro:if value="${baselink}">
-      <link name="fc">
-        <inertial>
-          <origin xyz="0 0 0" rpy="0 0 0"/>
-          <mass value="0.00001"/>
-          <inertia
-              ixx="0.000001" ixy="0.0" ixz="0.0"
-              iyy="0.000001" iyz="0.0"
-              izz="0.000002"/>
-        </inertial>
-      </link>
-      <joint name="fc_joint" type="fixed">
-        <child link="fc"/>
-        <parent link="link${self}"/>
-        <origin rpy="0 0 0" xyz="0.316 -0.004 0.043"/>
         <axis xyz="0 0 1"/>
       </joint>
