Commit message: [hydrus][tail] add servo config and link in urdf

File: robots/hydrus/robots/quad/tilt_10deg_15inch_livox_202505/robot.urdf.xacro (robot description, xacro)
@@ -52,3 +52,49 @@
     </inertial>
   </xacro:extra_module>
+  <!-- 3 tail -->
+  <link name="tail_link1"/>
+  <link name="tail_link2"/>
+  <link name="tail_link3"/>
+  <link name="tail_link4"/>
+  <link name="tail_link5"/>
+  <joint name="tail_joint1" type="revolute">
+    <limit effort="10.0" lower="${-pi/2}" upper="${pi/2}" velocity="0.5"/>
+    <parent link="link4"/>
+    <child link="tail_link1"/>
+    <origin xyz="0 0 0.5" rpy="0 0 0"/>
+    <axis xyz="0 0 1"/>
+    <dynamics damping="0.9" friction="0.05"/>
+  </joint>
+  <joint name="tail_joint2" type="revolute">
+    <limit effort="10.0" lower="${-pi/2}" upper="${pi/2}" velocity="0.5"/>
+    <parent link="tail_link1"/>
+    <child link="tail_link2"/>
+    <origin xyz="0 0 0" rpy="0 0 0"/>
+    <axis xyz="0 0 1"/>
+    <dynamics damping="0.9" friction="0.05"/>
+  </joint>
+  <joint name="tail_joint3" type="revolute">
+    <limit effort="10.0" lower="${-pi/2}" upper="${pi/2}" velocity="0.5"/>
+    <parent link="tail_link2"/>
+    <child link="tail_link3"/>
+    <origin xyz="0 0 0" rpy="0 0 0"/>
+    <axis xyz="0 0 1"/>
+    <dynamics damping="0.9" friction="0.05"/>
+  </joint>
+  <joint name="tail_joint4" type="revolute">
+    <limit effort="10.0" lower="${-pi/2}" upper="${pi/2}" velocity="0.5"/>
+    <parent link="tail_link3"/>
+    <child link="tail_link4"/>
+    <origin xyz="0 0 0" rpy="0 0 0"/>
+    <axis xyz="0 0 1"/>
+    <dynamics damping="0.9" friction="0.05"/>
+  </joint>
+  <joint name="tail_joint5" type="revolute">
+    <limit effort="10.0" lower="${-pi/2}" upper="${pi/2}" velocity="0.5"/>
+    <parent link="tail_link4"/>
+    <child link="tail_link5"/>
+    <origin xyz="0 0 0" rpy="0 0 0"/>
+    <axis xyz="0 0 1"/>
+    <dynamics damping="0.9" friction="0.05"/>
+  </joint>
 </robot>
