Commit message: [gimbalrotor][grape] update urdf to run simulation in gazebo

File: robots/gimbalrotor/urdf/grape/common.xacro (robot description, xacro)
@@ -6,3 +6,13 @@
   <thrust_link name="thrust" />
   <m_f_rate value="-0.0172" /> <!-- drug torque rate -->
+  <xacro:macro name="virtual_inertial" params="x:=0 y:=0 z:=0">
+    <inertial>
+      <origin xyz="${x} ${y} ${z}"/>
+      <mass value="0.00001"/>
+      <inertia
+          ixx="0.000001" ixy="0.0" ixz="0.0"
+          iyy="0.000001" iyz="0.0"
+          izz="0.000002"/>
+    </inertial>
+  </xacro:macro>
 </robot>

File: robots/gimbalrotor/urdf/grape/gimbalrotor.urdf.xacro (robot description, xacro)
@@ -1,4 +1,5 @@
 <?xml version='1.0' encoding='UTF-8'?>
 <robot name="gimbalrotor" xmlns:xacro="http://www.ros.org/wiki/xacro">
+  <xacro:include filename="$(find gimbalrotor)/urdf/grape/common.xacro"/>
   <link name="root">
     <inertial>
@@ -226,6 +227,42 @@
     <!-- </collision> -->
   </link>
+  <link name="rotor_arm1">
+    <xacro:virtual_inertial/>
+  </link>
+  <link name="rotor_arm2">
+    <xacro:virtual_inertial/>
+  </link>
+  <link name="rotor_arm3">
+    <xacro:virtual_inertial/>
+  </link>
+  <link name="rotor_arm4">
+    <xacro:virtual_inertial/>
+  </link>
+  <joint name="rotor_arm1_joint" type="fixed">
+    <parent link="main_body"/>
+    <child link="rotor_arm1"/>
+    <axis xyz="0 0 1"/>
+    <origin xyz="-0.22309 -0.22309 0.0" rpy="0.0 -0.0 -2.3562"/>
+  </joint>
+  <joint name="rotor_arm2_joint" type="fixed">
+    <parent link="main_body"/>
+    <child link="rotor_arm2"/>
+    <axis xyz="0 0 1"/>
+    <origin xyz="0.22309 -0.22309 0.0" rpy="-0.0 -0.0 -0.7854000000000001"/>
+  </joint>
+  <joint name="rotor_arm3_joint" type="fixed">
+    <parent link="main_body"/>
+    <child link="rotor_arm3"/>
+    <axis xyz="0 0 1"/>
+    <origin xyz="0.22309 0.22309 0.0" rpy="0.0 -0.0 0.7854000000000001"/>
+  </joint>
+  <joint name="rotor_arm4_joint" type="fixed">
+    <parent link="main_body"/>
+    <child link="rotor_arm4"/>
+    <axis xyz="0 0 1"/>
+    <origin xyz="-0.22309 0.22309 0.0" rpy="0.0 -0.0 2.3562"/>
+  </joint>
   <joint name="gimbal1" type="revolute">
-    <limit effort="0.0" velocity="0.0" lower="-3.14" upper="3.14"/>
+    <limit effort="5.0" velocity="10.0" lower="-3.14" upper="3.14"/>
     <parent link="main_body"/>
     <child link="gimbal1_link"/>
@@ -234,5 +271,5 @@
   </joint>
   <joint name="rotor1" type="continuous">
-    <limit effort="0.0" velocity="0.0"/>
+    <limit effort="0.0" velocity="0.0" lower="0.0" upper="30.0"/>
     <parent link="gimbal1_link"/>
     <child link="thrust1"/>
@@ -241,5 +278,5 @@
   </joint>
   <joint name="gimbal2" type="revolute">
-    <limit effort="0.0" velocity="0.0" lower="-3.14" upper="3.14"/>
+    <limit effort="5.0" velocity="10.0" lower="-3.14" upper="3.14"/>
     <parent link="main_body"/>
     <child link="gimbal2_link"/>
@@ -248,5 +285,5 @@
   </joint>
   <joint name="rotor2" type="continuous">
-    <limit effort="0.0" velocity="0.0"/>
+    <limit effort="0.0" velocity="0.0" lower="0.0" upper="30.0"/>
     <parent link="gimbal2_link"/>
     <child link="thrust2"/>
@@ -255,5 +292,5 @@
   </joint>
   <joint name="gimbal3" type="revolute">
-    <limit effort="0.0" velocity="0.0" lower="-3.14" upper="3.14"/>
+    <limit effort="5.0" velocity="10.0" lower="-3.14" upper="3.14"/>
     <parent link="main_body"/>
     <child link="gimbal3_link"/>
@@ -262,5 +299,5 @@
   </joint>
   <joint name="rotor3" type="continuous">
-    <limit effort="0.0" velocity="0.0"/>
+    <limit effort="0.0" velocity="0.0" lower="0.0" upper="30.0"/>
     <parent link="gimbal3_link"/>
     <child link="thrust3"/>
@@ -269,5 +306,5 @@
   </joint>
   <joint name="gimbal4" type="revolute">
-    <limit effort="0.0" velocity="0.0" lower="-3.14" upper="3.14"/>
+    <limit effort="5.0" velocity="10.0" lower="-3.14" upper="3.14"/>
     <parent link="main_body"/>
     <child link="gimbal4_link"/>
@@ -276,5 +313,5 @@
   </joint>
   <joint name="rotor4" type="continuous">
-    <limit effort="0.0" velocity="0.0"/>
+    <limit effort="0.0" velocity="0.0" lower="0.0" upper="30.0"/>
     <parent link="gimbal4_link"/>
     <child link="thrust4"/>
@@ -322,4 +359,44 @@
     </actuator>
   </transmission>
+    <transmission name="rotor_tran1">
+      <type>transmission_interface/SimpleTransmission</type>
+      <joint name="rotor1">
+        <hardwareInterface>RotorInterface</hardwareInterface>
+      </joint>
+      <actuator name="rotor_actuator1">
+        <hardwareInterface>RotorInterface</hardwareInterface>
+        <mechanicalReduction>1</mechanicalReduction>
+      </actuator>
+    </transmission>
+    <transmission name="rotor_tran2">
+      <type>transmission_interface/SimpleTransmission</type>
+      <joint name="rotor2">
+        <hardwareInterface>RotorInterface</hardwareInterface>
+      </joint>
+      <actuator name="rotor_actuator2">
+        <hardwareInterface>RotorInterface</hardwareInterface>
+        <mechanicalReduction>1</mechanicalReduction>
+      </actuator>
+    </transmission>
+    <transmission name="rotor_tran3">
+      <type>transmission_interface/SimpleTransmission</type>
+      <joint name="rotor3">
+        <hardwareInterface>RotorInterface</hardwareInterface>
+      </joint>
+      <actuator name="rotor_actuator3">
+        <hardwareInterface>RotorInterface</hardwareInterface>
+        <mechanicalReduction>1</mechanicalReduction>
+      </actuator>
+    </transmission>
+    <transmission name="rotor_tran4">
+      <type>transmission_interface/SimpleTransmission</type>
+      <joint name="rotor4">
+        <hardwareInterface>RotorInterface</hardwareInterface>
+      </joint>
+      <actuator name="rotor_actuator4">
+        <hardwareInterface>RotorInterface</hardwareInterface>
+        <mechanicalReduction>1</mechanicalReduction>
+      </actuator>
+    </transmission>
   <material name="__unnamed_material_1">
     <color rgba="0.10980392 0.10980392 0.10980392 1.        "/>
