Commit message: [grape] add lidar urdf to arm model

File: robots/gimbalrotor/urdf/grape/gimbalrotor_with_arm.urdf.xacro (robot description, xacro)
@@ -35,4 +35,20 @@
     <axis xyz="0 0 1"/>
   </joint>
+  <link name="lidar_imu">
+    <inertial>
+      <origin xyz="0 0 0" rpy="0 0 0"/>
+      <mass value="0.00001"/>
+      <inertia
+          ixx="0.000001" ixy="0.0" ixz="0.0"
+          iyy="0.000001" iyz="0.0"
+          izz="0.000001"/>
+    </inertial>
+  </link>
+  <joint name="lidar_joint" type="fixed">
+    <child link="lidar_imu"/>
+    <parent link="main_body"/>
+    <origin xyz="0 0 -0.08" rpy="3.14159 0 0"/>
+    <axis xyz="0 0 1"/>
+  </joint>
   <link name="main_body">
     <inertial>
