Commit message: update arm urdf

File: robots/gimbalrotor/urdf/grape/gimbalrotor_with_arm.urdf (robot description, URDF)
Before this commit: robot gimbalrotor_with_arm, 39 links, 38 joints
Joints:
- joint arm_joint2_joint1: limit lower=-0.567 upper=0.567 effort=0.0 velocity=0.0 -> lower=-3.14159 upper=3.14159 effort=0.0 velocity=0.0
- joint arm_joint3_joint1: limit lower=-0.567 upper=0.567 effort=0.0 velocity=0.0 -> lower=-3.14159 upper=3.14159 effort=0.0 velocity=0.0
- joint arm_joint4_joint1: limit lower=-0.567 upper=0.567 effort=0.0 velocity=0.0 -> lower=-3.14159 upper=3.14159 effort=0.0 velocity=0.0
