Commit message: [gimbalrotor][grape] update urdf

File: robots/gimbalrotor/urdf/grape/gimbalrotor.urdf.xacro (robot description, xacro)
@@ -1,13 +1,45 @@
 <?xml version='1.0' encoding='UTF-8'?>
 <robot name="gimbalrotor" xmlns:xacro="http://www.ros.org/wiki/xacro">
+  <link name="root">
+    <inertial>
+      <origin xyz="0 0 0" rpy="0 0 0"/>
+      <mass value="0.00001"/>
+      <inertia
+          ixx="0.000001" ixy="0.0" ixz="0.0"
+          iyy="0.000001" iyz="0.0"
+          izz="0.000001"/>
+    </inertial>
+  </link>
+  <joint name="root_joint" type="fixed">
+    <parent link="root"/>
+    <child link="main_body"/>
+    <origin rpy="0 0 0" xyz="0 0 0"/>
+    <axis xyz="0 0 1"/>
+  </joint>
+  <link name="fc">
+    <inertial>
+      <origin xyz="0 0 0" rpy="0 0 0"/>
+      <mass value="0.00001"/>
+      <inertia
+          ixx="0.000001" ixy="0.0" ixz="0.0"
+          iyy="0.000001" iyz="0.0"
+          izz="0.000001"/>
+    </inertial>
+  </link>
+  <joint name="fc_joint" type="fixed">
+    <child link="fc"/>
+    <parent link="main_body"/>
+    <origin rpy="0 0 0" xyz="0 0 0"/>
+    <axis xyz="0 0 1"/>
+  </joint>
   <link name="main_body">
     <inertial>
-      <!-- <origin xyz="-0.00202460418348044 -0.000510481706680737 -0.0123651551887967" rpy="0.0 -0.0 0.0"/> -->
-      <!-- <mass value="1.40071559053294"/> -->
-      <!-- <inertia ixx="0.00167259281385339" ixy="-1.88191851673578e-07" ixz="7.17787328777675e-07" iyy="0.00167984573863287" iyz="4.03619596691479e-08" izz="0.00304193991451692"/> -->
-    </inertial>
-    <visual>
-      <geometry>
-        <mesh filename="package://gimbalrotor/grape/meshes/main_body.dae"/>
+      <origin xyz="-0.00202460418348044 -0.000510481706680737 -0.0123651551887967" rpy="0.0 -0.0 0.0"/>
+      <mass value="1.40071559053294"/>
+      <inertia ixx="0.00167259281385339" ixy="-1.88191851673578e-07" ixz="7.17787328777675e-07" iyy="0.00167984573863287" iyz="4.03619596691479e-08" izz="0.00304193991451692"/>
+    </inertial>
+    <visual>
+      <geometry>
+        <mesh filename="package://gimbalrotor/urdf/grape/meshes/main_body.dae"/>
       </geometry>
       <material name="__unnamed_material_1"/>
@@ -16,5 +48,6 @@
     <collision>
       <geometry>
-        <mesh filename="package://gimbalrotor/grape/meshes/main_body.stl"/>
+        <!-- <mesh filename="package://gimbalrotor/urdf/grape/meshes/main_body.stl"/> -->
+        <box size="0.25 0.25 0.035"/>
       </geometry>
       <origin xyz="0.0 0.0 0.0" rpy="0.0 -0.0 0.0"/>
@@ -32,15 +65,15 @@
     <visual>
       <geometry>
-        <mesh filename="package://gimbalrotor/grape/meshes/gimbal1_link.dae"/>
+        <mesh filename="package://gimbalrotor/urdf/grape/meshes/gimbal1_link.dae"/>
       </geometry>
       <material name="__unnamed_material_2"/>
       <origin xyz="0.0 0.0 0.0" rpy="0.0 -0.0 0.0"/>
     </visual>
-    <collision>
-      <geometry>
-        <mesh filename="package://gimbalrotor/grape/meshes/gimbal1_link.stl"/>
-      </geometry>
-      <origin xyz="0.0 0.0 0.0" rpy="0.0 -0.0 0.0"/>
-    </collision>
+    <!-- <collision> -->
+      <!-- <geometry> -->
+      <!--   <mesh filename="package://gimbalrotor/urdf/grape/meshes/gimbal1_link.stl"/> -->
+      <!-- </geometry> -->
+      <!-- <origin xyz="0.0 0.0 0.0" rpy="0.0 -0.0 0.0"/> -->
+    <!-- </collision> -->
   </link>
   <link name="thrust1">
@@ -52,15 +85,15 @@
     <visual>
       <geometry>
-        <mesh filename="package://gimbalrotor/grape/meshes/thrust1.dae"/>
+        <mesh filename="package://gimbalrotor/urdf/grape/meshes/thrust1.dae"/>
       </geometry>
       <material name="__unnamed_material_3"/>
       <origin xyz="0.0 0.0 0.0" rpy="0.0 -0.0 0.0"/>
     </visual>
-    <collision>
-      <geometry>
-        <mesh filename="package://gimbalrotor/grape/meshes/thrust1.stl"/>
-      </geometry>
-      <origin xyz="0.0 0.0 0.0" rpy="0.0 -0.0 0.0"/>
-    </collision>
+    <!-- <collision> -->
+      <!-- <geometry> -->
+      <!--   <mesh filename="package://gimbalrotor/urdf/grape/meshes/thrust1.stl"/> -->
+      <!-- </geometry> -->
+      <!-- <origin xyz="0.0 0.0 0.0" rpy="0.0 -0.0 0.0"/> -->
+    <!-- </collision> -->
   </link>
   <link name="gimbal2_link">
@@ -75,15 +108,15 @@
     <visual>
       <geometry>
-        <mesh filename="package://gimbalrotor/grape/meshes/gimbal2_link.dae"/>
+        <mesh filename="package://gimbalrotor/urdf/grape/meshes/gimbal2_link.dae"/>
       </geometry>
       <material name="__unnamed_material_4"/>
       <origin xyz="0.0 0.0 0.0" rpy="0.0 -0.0 0.0"/>
     </visual>
-    <collision>
-      <geometry>
-        <mesh filename="package://gimbalrotor/grape/meshes/gimbal2_link.stl"/>
-      </geometry>
-      <origin xyz="0.0 0.0 0.0" rpy="0.0 -0.0 0.0"/>
-    </collision>
+    <!-- <collision> -->
+    <!--   <geometry> -->
+    <!--     <mesh filename="package://gimbalrotor/urdf/grape/meshes/gimbal2_link.stl"/> -->
+    <!--   </geometry> -->
+    <!--   <origin xyz="0.0 0.0 0.0" rpy="0.0 -0.0 0.0"/> -->
+    <!-- </collision> -->
   </link>
   <link name="thrust2">
@@ -95,15 +128,15 @@
     <visual>
       <geometry>
-        <mesh filename="package://gimbalrotor/grape/meshes/thrust2.dae"/>
+        <mesh filename="package://gimbalrotor/urdf/grape/meshes/thrust2.dae"/>
       </geometry>
       <material name="__unnamed_material_5"/>
       <origin xyz="0.0 0.0 0.0" rpy="0.0 -0.0 0.0"/>
     </visual>
-    <collision>
-      <geometry>
-        <mesh filename="package://gimbalrotor/grape/meshes/thrust2.stl"/>
-      </geometry>
-      <origin xyz="0.0 0.0 0.0" rpy="0.0 -0.0 0.0"/>
-    </collision>
+    <!-- <collision> -->
+    <!--   <geometry> -->
+    <!--     <mesh filename="package://gimbalrotor/urdf/grape/meshes/thrust2.stl"/> -->
+    <!--   </geometry> -->
+    <!--   <origin xyz="0.0 0.0 0.0" rpy="0.0 -0.0 0.0"/> -->
+    <!-- </collision> -->
   </link>
   <link name="gimbal3_link">
@@ -118,15 +151,15 @@
     <visual>
       <geometry>
-        <mesh filename="package://gimbalrotor/grape/meshes/gimbal3_link.dae"/>
+        <mesh filename="package://gimbalrotor/urdf/grape/meshes/gimbal3_link.dae"/>
       </geometry>
       <material name="__unnamed_material_6"/>
       <origin xyz="0.0 0.0 0.0" rpy="0.0 -0.0 0.0"/>
     </visual>
-    <collision>
-      <geometry>
-        <mesh filename="package://gimbalrotor/grape/meshes/gimbal3_link.stl"/>
-      </geometry>
-      <origin xyz="0.0 0.0 0.0" rpy="0.0 -0.0 0.0"/>
-    </collision>
+    <!-- <collision> -->
+      <!-- <geometry> -->
+      <!--   <mesh filename="package://gimbalrotor/urdf/grape/meshes/gimbal3_link.stl"/> -->
+      <!-- </geometry> -->
+      <!-- <origin xyz="0.0 0.0 0.0" rpy="0.0 -0.0 0.0"/> -->
+    <!-- </collision> -->
   </link>
   <link name="thrust3">
@@ -138,15 +171,15 @@
     <visual>
       <geometry>
-        <mesh filename="package://gimbalrotor/grape/meshes/thrust3.dae"/>
+        <mesh filename="package://gimbalrotor/urdf/grape/meshes/thrust3.dae"/>
       </geometry>
       <material name="__unnamed_material_7"/>
       <origin xyz="0.0 0.0 0.0" rpy="0.0 -0.0 0.0"/>
     </visual>
-    <collision>
-      <geometry>
-        <mesh filename="package://gimbalrotor/grape/meshes/thrust3.stl"/>
-      </geometry>
-      <origin xyz="0.0 0.0 0.0" rpy="0.0 -0.0 0.0"/>
-    </collision>
+    <!-- <collision> -->
+      <!-- <geometry> -->
+      <!--   <mesh filename="package://gimbalrotor/urdf/grape/meshes/thrust3.stl"/> -->
+      <!-- </geometry> -->
+      <!-- <origin xyz="0.0 0.0 0.0" rpy="0.0 -0.0 0.0"/> -->
+    <!-- </collision> -->
   </link>
   <link name="gimbal4_link">
@@ -161,15 +194,15 @@
     <visual>
       <geometry>
-        <mesh filename="package://gimbalrotor/grape/meshes/gimbal4_link.dae"/>
+        <mesh filename="package://gimbalrotor/urdf/grape/meshes/gimbal4_link.dae"/>
       </geometry>
       <material name="__unnamed_material_8"/>
       <origin xyz="0.0 0.0 0.0" rpy="0.0 -0.0 0.0"/>
     </visual>
-    <collision>
-      <geometry>
-        <mesh filename="package://gimbalrotor/grape/meshes/gimbal4_link.stl"/>
-      </geometry>
-      <origin xyz="0.0 0.0 0.0" rpy="0.0 -0.0 0.0"/>
-    </collision>
+    <!-- <collision> -->
+      <!-- <geometry> -->
+      <!--   <mesh filename="package://gimbalrotor/urdf/grape/meshes/gimbal4_link.stl"/> -->
+      <!-- </geometry> -->
+      <!-- <origin xyz="0.0 0.0 0.0" rpy="0.0 -0.0 0.0"/> -->
+    <!-- </collision> -->
   </link>
   <link name="thrust4">
@@ -181,15 +214,15 @@
     <visual>
       <geometry>
-        <mesh filename="package://gimbalrotor/grape/meshes/thrust4.dae"/>
+        <mesh filename="package://gimbalrotor/urdf/grape/meshes/thrust4.dae"/>
       </geometry>
       <material name="__unnamed_material_9"/>
       <origin xyz="0.0 0.0 0.0" rpy="0.0 -0.0 0.0"/>
     </visual>
-    <collision>
-      <geometry>
-        <mesh filename="package://gimbalrotor/grape/meshes/thrust4.stl"/>
-      </geometry>
-      <origin xyz="0.0 0.0 0.0" rpy="0.0 -0.0 0.0"/>
-    </collision>
+    <!-- <collision> -->
+      <!-- <geometry> -->
+      <!--   <mesh filename="package://gimbalrotor/urdf/grape/meshes/thrust4.stl"/> -->
+      <!-- </geometry> -->
+      <!-- <origin xyz="0.0 0.0 0.0" rpy="0.0 -0.0 0.0"/> -->
+    <!-- </collision> -->
   </link>
   <joint name="gimbal1" type="revolute">
@@ -249,4 +282,44 @@
     <origin xyz="0.0 0.0 0.0585" rpy="0.0 -0.0 0.0"/>
   </joint>
+  <transmission name="gimbal1_tran">
+    <type>transmission_interface/SimpleTransmission</type>
+    <joint name="gimbal1">
+      <hardwareInterface>hardware_interface/EffortJointInterface</hardwareInterface>
+    </joint>
+    <actuator name="servo1">
+      <hardwareInterface>hardware_interface/EffortJointInterface</hardwareInterface>
+      <mechanicalReduction>1</mechanicalReduction>
+    </actuator>
+  </transmission>
+  <transmission name="gimbal2_tran">
+    <type>transmission_interface/SimpleTransmission</type>
+    <joint name="gimbal2">
+      <hardwareInterface>hardware_interface/EffortJointInterface</hardwareInterface>
+    </joint>
+    <actuator name="servo2">
+      <hardwareInterface>hardware_interface/EffortJointInterface</hardwareInterface>
+      <mechanicalReduction>1</mechanicalReduction>
+    </actuator>
+  </transmission>
+  <transmission name="gimbal3_tran">
+    <type>transmission_interface/SimpleTransmission</type>
+    <joint name="gimbal3">
+      <hardwareInterface>hardware_interface/EffortJointInterface</hardwareInterface>
+    </joint>
+    <actuator name="servo3">
+      <hardwareInterface>hardware_interface/EffortJointInterface</hardwareInterface>
+      <mechanicalReduction>1</mechanicalReduction>
+    </actuator>
+  </transmission>
+  <transmission name="gimbal4_tran">
+    <type>transmission_interface/SimpleTransmission</type>
+    <joint name="gimbal4">
+      <hardwareInterface>hardware_interface/EffortJointInterface</hardwareInterface>
+    </joint>
+    <actuator name="servo4">
+      <hardwareInterface>hardware_interface/EffortJointInterface</hardwareInterface>
+      <mechanicalReduction>1</mechanicalReduction>
+    </actuator>
+  </transmission>
   <material name="__unnamed_material_1">
     <color rgba="0.10980392 0.10980392 0.10980392 1.        "/>

Commit message: update grape urdf

File: robots/gimbalrotor/urdf/grape/gimbalrotor.urdf.xacro (robot description, xacro)
@@ -36,7 +36,10 @@
   <link name="main_body">
     <inertial>
-      <origin xyz="-0.00202460418348044 -0.000510481706680737 -0.0123651551887967" rpy="0.0 -0.0 0.0"/>
-      <mass value="1.40071559053294"/>
-      <inertia ixx="0.00167259281385339" ixy="-1.88191851673578e-07" ixz="7.17787328777675e-07" iyy="0.00167984573863287" iyz="4.03619596691479e-08" izz="0.00304193991451692"/>
+      <origin xyz="-0.0041019 0.0000721 -0.0183334" rpy="0.0 -0.0 0.0"/>
+      <mass value="1.3193189"/>
+      <inertia ixx="0.0150906" ixy="-0.0000095" ixz="-0.0001112" iyy="0.0153469" iyz="-0.0000102" izz="0.0122100"/>
+      <!-- <origin xyz="-0.00202460418348044 -0.000510481706680737 -0.0123651551887967" rpy="0.0 -0.0 0.0"/> -->
+      <!-- <mass value="1.40071559053294"/> -->
+      <!-- <inertia ixx="0.00167259281385339" ixy="-1.88191851673578e-07" ixz="7.17787328777675e-07" iyy="0.00167984573863287" iyz="4.03619596691479e-08" izz="0.00304193991451692"/> -->
     </inertial>
     <visual>
@@ -57,7 +60,7 @@
   <link name="gimbal1_link">
     <inertial>
-      <origin xyz="-0.00926567494919711 1.9703972765894e-06 0.0128616849753725" rpy="0.0 -0.0 0.0"/>
-      <mass value="0.243868409767181"/>
-      <inertia ixx="4.70366622152039e-05" ixy="-5.23334464430229e-09" ixz="-4.58510270196035e-07" iyy="4.49457729860046e-05" iyz="-2.62506744960952e-09" izz="4.59133399019853e-05"/>
+      <origin xyz="0.0097185 -0.0000023 0.0115030" rpy="0.0 -0.0 0.0"/>
+      <mass value="0.2647482"/>
+      <inertia ixx="0.0004342" ixy="0.0000000" ixz="-0.0000960" iyy="0.0005399" iyz="0.0000000" izz="0.0001644"/>
       <!-- <origin xyz="-0.00926567494919711 1.9703972765894e-06 0.0128616849753725" rpy="0.0 -0.0 0.0"/> -->
       <!-- <mass value="0.243868409767181"/> -->
@@ -100,7 +103,7 @@
   <link name="gimbal2_link">
     <inertial>
-      <origin xyz="-0.00926567494919772 1.97039712329184e-06 0.0128616849753724" rpy="0.0 -0.0 0.0"/>
-      <mass value="0.243868409767181"/>
-      <inertia ixx="4.70366622152039e-05" ixy="-5.23334464430183e-09" ixz="-4.5851027019603e-07" iyy="4.49457729860046e-05" iyz="-2.62506744960961e-09" izz="4.59133399019854e-05"/>
+      <origin xyz="0.0097185 -0.0000023 0.0115030" rpy="0.0 -0.0 0.0"/>
+      <mass value="0.2647482"/>
+      <inertia ixx="0.0004342" ixy="0.0000000" ixz="-0.0000960" iyy="0.0005399" iyz="0.0000000" izz="0.0001644"/>
       <!-- <origin xyz="-0.00926567494919767 1.97039727626247e-06 0.0128616849753725" rpy="0.0 -0.0 0.0"/> -->
       <!-- <mass value="0.243868409767181"/> -->
@@ -143,7 +146,7 @@
   <link name="gimbal3_link">
     <inertial>
-      <origin xyz="-0.00926567494919772 1.97039712329184e-06 0.0128616849753724" rpy="0.0 -0.0 0.0"/>
-      <mass value="0.243868409767181"/>
-      <inertia ixx="4.70366622152039e-05" ixy="-5.23334464430183e-09" ixz="-4.5851027019603e-07" iyy="4.49457729860046e-05" iyz="-2.62506744960961e-09" izz="4.59133399019854e-05"/>
+      <origin xyz="0.0097185 -0.0000023 0.0115030" rpy="0.0 -0.0 0.0"/>
+      <mass value="0.2647482"/>
+      <inertia ixx="0.0004342" ixy="0.0000000" ixz="-0.0000960" iyy="0.0005399" iyz="0.0000000" izz="0.0001644"/>
       <!-- <origin xyz="-0.00926567494919739 1.97039727626326e-06 0.0128616849753725" rpy="0.0 -0.0 0.0"/> -->
       <!-- <mass value="0.243868409767181"/> -->
@@ -186,7 +189,7 @@
   <link name="gimbal4_link">
     <inertial>
-      <origin xyz="-0.00926567494919772 1.97039712329184e-06 0.0128616849753724" rpy="0.0 -0.0 0.0"/>
-      <mass value="0.243868409767181"/>
-      <inertia ixx="4.70366622152039e-05" ixy="-5.23334464430183e-09" ixz="-4.5851027019603e-07" iyy="4.49457729860046e-05" iyz="-2.62506744960961e-09" izz="4.59133399019854e-05"/>
+      <origin xyz="0.0097185 -0.0000023 0.0115030" rpy="0.0 -0.0 0.0"/>
+      <mass value="0.2647482"/>
+      <inertia ixx="0.0004342" ixy="0.0000000" ixz="-0.0000960" iyy="0.0005399" iyz="0.0000000" izz="0.0001644"/>
       <!-- <origin xyz="-0.00926567494919772 1.97039712329184e-06 0.0128616849753724" rpy="0.0 -0.0 0.0"/> -->
       <!-- <mass value="0.243868409767181"/> -->

Commit message: [gimbalrotor][grape] remove comment in urdf

File: robots/gimbalrotor/urdf/grape/gimbalrotor.urdf.xacro (robot description, xacro)
@@ -39,7 +39,4 @@
       <mass value="1.3193189"/>
       <inertia ixx="0.0150906" ixy="-0.0000095" ixz="-0.0001112" iyy="0.0153469" iyz="-0.0000102" izz="0.0122100"/>
-      <!-- <origin xyz="-0.00202460418348044 -0.000510481706680737 -0.0123651551887967" rpy="0.0 -0.0 0.0"/> -->
-      <!-- <mass value="1.40071559053294"/> -->
-      <!-- <inertia ixx="0.00167259281385339" ixy="-1.88191851673578e-07" ixz="7.17787328777675e-07" iyy="0.00167984573863287" iyz="4.03619596691479e-08" izz="0.00304193991451692"/> -->
     </inertial>
     <visual>
@@ -63,7 +60,4 @@
       <mass value="0.2647482"/>
       <inertia ixx="0.0004342" ixy="0.0000000" ixz="-0.0000960" iyy="0.0005399" iyz="0.0000000" izz="0.0001644"/>
-      <!-- <origin xyz="-0.00926567494919711 1.9703972765894e-06 0.0128616849753725" rpy="0.0 -0.0 0.0"/> -->
-      <!-- <mass value="0.243868409767181"/> -->
-      <!-- <inertia ixx="4.70366622152039e-05" ixy="-5.23334464430229e-09" ixz="-4.58510270196035e-07" iyy="4.49457729860046e-05" iyz="-2.62506744960952e-09" izz="4.59133399019853e-05"/> -->
     </inertial>
     <visual>
@@ -106,7 +100,4 @@
       <mass value="0.2647482"/>
       <inertia ixx="0.0004342" ixy="0.0000000" ixz="-0.0000960" iyy="0.0005399" iyz="0.0000000" izz="0.0001644"/>
-      <!-- <origin xyz="-0.00926567494919767 1.97039727626247e-06 0.0128616849753725" rpy="0.0 -0.0 0.0"/> -->
-      <!-- <mass value="0.243868409767181"/> -->
-      <!-- <inertia ixx="4.70366622152039e-05" ixy="-5.23334464430243e-09" ixz="-4.58510270196032e-07" iyy="4.49457729860046e-05" iyz="-2.62506744960964e-09" izz="4.59133399019854e-05"/> -->
     </inertial>
     <visual>
@@ -149,7 +140,4 @@
       <mass value="0.2647482"/>
       <inertia ixx="0.0004342" ixy="0.0000000" ixz="-0.0000960" iyy="0.0005399" iyz="0.0000000" izz="0.0001644"/>
-      <!-- <origin xyz="-0.00926567494919739 1.97039727626326e-06 0.0128616849753725" rpy="0.0 -0.0 0.0"/> -->
-      <!-- <mass value="0.243868409767181"/> -->
-      <!-- <inertia ixx="4.70366622152039e-05" ixy="-5.23334464430207e-09" ixz="-4.58510270196014e-07" iyy="4.49457729860046e-05" iyz="-2.62506744960844e-09" izz="4.59133399019853e-05"/> -->
     </inertial>
     <visual>
@@ -192,7 +180,4 @@
       <mass value="0.2647482"/>
       <inertia ixx="0.0004342" ixy="0.0000000" ixz="-0.0000960" iyy="0.0005399" iyz="0.0000000" izz="0.0001644"/>
-      <!-- <origin xyz="-0.00926567494919772 1.97039712329184e-06 0.0128616849753724" rpy="0.0 -0.0 0.0"/> -->
-      <!-- <mass value="0.243868409767181"/> -->
-      <!-- <inertia ixx="4.70366622152039e-05" ixy="-5.23334464430183e-09" ixz="-4.5851027019603e-07" iyy="4.49457729860046e-05" iyz="-2.62506744960961e-09" izz="4.59133399019854e-05"/> -->
     </inertial>
     <visual>

Commit message: [gimbalrotor][grape] use stl for urdf visual to avoid crash of gazebo gui

File: robots/gimbalrotor/urdf/grape/gimbalrotor.urdf.xacro (robot description, xacro)
@@ -42,5 +42,5 @@
     <visual>
       <geometry>
-        <mesh filename="package://gimbalrotor/urdf/grape/meshes/main_body.dae"/>
+        <mesh filename="package://gimbalrotor/urdf/grape/meshes/main_body.stl"/>
       </geometry>
       <material name="__unnamed_material_1"/>
@@ -63,5 +63,5 @@
     <visual>
       <geometry>
-        <mesh filename="package://gimbalrotor/urdf/grape/meshes/gimbal1_link.dae"/>
+        <mesh filename="package://gimbalrotor/urdf/grape/meshes/gimbal1_link.stl"/>
       </geometry>
       <material name="__unnamed_material_2"/>
@@ -83,5 +83,5 @@
     <visual>
       <geometry>
-        <mesh filename="package://gimbalrotor/urdf/grape/meshes/thrust1.dae"/>
+        <mesh filename="package://gimbalrotor/urdf/grape/meshes/thrust1.stl"/>
       </geometry>
       <material name="__unnamed_material_3"/>
@@ -103,5 +103,5 @@
     <visual>
       <geometry>
-        <mesh filename="package://gimbalrotor/urdf/grape/meshes/gimbal2_link.dae"/>
+        <mesh filename="package://gimbalrotor/urdf/grape/meshes/gimbal2_link.stl"/>
       </geometry>
       <material name="__unnamed_material_4"/>
@@ -123,5 +123,5 @@
     <visual>
       <geometry>
-        <mesh filename="package://gimbalrotor/urdf/grape/meshes/thrust2.dae"/>
+        <mesh filename="package://gimbalrotor/urdf/grape/meshes/thrust2.stl"/>
       </geometry>
       <material name="__unnamed_material_5"/>
@@ -143,5 +143,5 @@
     <visual>
       <geometry>
-        <mesh filename="package://gimbalrotor/urdf/grape/meshes/gimbal3_link.dae"/>
+        <mesh filename="package://gimbalrotor/urdf/grape/meshes/gimbal3_link.stl"/>
       </geometry>
       <material name="__unnamed_material_6"/>
@@ -163,5 +163,5 @@
     <visual>
       <geometry>
-        <mesh filename="package://gimbalrotor/urdf/grape/meshes/thrust3.dae"/>
+        <mesh filename="package://gimbalrotor/urdf/grape/meshes/thrust3.stl"/>
       </geometry>
       <material name="__unnamed_material_7"/>
@@ -183,5 +183,5 @@
     <visual>
       <geometry>
-        <mesh filename="package://gimbalrotor/urdf/grape/meshes/gimbal4_link.dae"/>
+        <mesh filename="package://gimbalrotor/urdf/grape/meshes/gimbal4_link.stl"/>
       </geometry>
       <material name="__unnamed_material_8"/>
@@ -203,5 +203,5 @@
     <visual>
       <geometry>
-        <mesh filename="package://gimbalrotor/urdf/grape/meshes/thrust4.dae"/>
+        <mesh filename="package://gimbalrotor/urdf/grape/meshes/thrust4.stl"/>
       </geometry>
       <material name="__unnamed_material_9"/>

Commit message: [gimbalrotor][grape] enable to use livox and fastlio

File: robots/gimbalrotor/urdf/grape/gimbalrotor.urdf.xacro (robot description, xacro)
@@ -34,4 +34,20 @@
     <axis xyz="0 0 1"/>
   </joint>
+  <link name="lidar_imu">
+    <inertial>
+      <origin xyz="0 0 0" rpy="0 0 0"/>
+      <mass value="0.00001"/>
+      <inertia
+          ixx="0.000001" ixy="0.0" ixz="0.0"
+          iyy="0.000001" iyz="0.0"
+          izz="0.000001"/>
+    </inertial>
+  </link>
+  <joint name="lidar_joint" type="fixed">
+    <child link="lidar_imu"/>
+    <parent link="main_body"/>
+    <origin xyz="0 0 0.08" rpy="0 0 0"/>
+    <axis xyz="0 0 1"/>
+  </joint>
   <link name="main_body">
     <inertial>

Commit message: [grape] update lidar frame

File: robots/gimbalrotor/urdf/grape/gimbalrotor.urdf.xacro (robot description, xacro)
@@ -47,5 +47,5 @@
     <child link="lidar_imu"/>
     <parent link="main_body"/>
-    <origin xyz="0 0 0.08" rpy="0 0 0"/>
+    <origin xyz="0 0 -0.08" rpy="3.14159 0 0"/>
     <axis xyz="0 0 1"/>
   </joint>

Commit message: [grape] add battery link to urdf

File: robots/gimbalrotor/urdf/grape/gimbalrotor.urdf.xacro (robot description, xacro)
@@ -50,4 +50,20 @@
     <axis xyz="0 0 1"/>
   </joint>
+  <link name="battery">
+    <inertial>
+      <origin xyz="0 0 0" rpy="0 0 0"/>
+      <mass value="1.1"/>
+      <inertia
+          ixx="0.0012" ixy="0.0" ixz="0.0"
+          iyy="0.0012" iyz="0.0"
+          izz="0.0012"/>
+    </inertial>
+  </link>
+  <joint name="battery_joint" type="fixed">
+    <parent link="main_body"/>
+    <child link="battery"/>
+    <origin xyz="0 0 -0.08" rpy="3.14159 0 0"/>
+    <axis xyz="0 0 1"/>
+  </joint>
   <link name="main_body">
     <inertial>
