Commit message: [gimbalrotor][grape] add gimbal angle limits for grape for safety

File: robots/gimbalrotor/urdf/grape/gimbalrotor.urdf.xacro (robot description, xacro)
@@ -207,5 +207,5 @@
   </link>
   <joint name="gimbal1" type="revolute">
-    <limit effort="1.5" velocity="6.0" lower="-3.14" upper="3.14"/>
+    <limit effort="1.5" velocity="6.0" lower="-1.0" upper="1.0"/>
     <parent link="main_body"/>
     <child link="gimbal1_link"/>
@@ -221,5 +221,5 @@
   </joint>
   <joint name="gimbal2" type="revolute">
-    <limit effort="1.5" velocity="6.0" lower="-3.14" upper="3.14"/>
+    <limit effort="1.5" velocity="6.0" lower="-1.0" upper="1.0"/>
     <parent link="main_body"/>
     <child link="gimbal2_link"/>
@@ -235,5 +235,5 @@
   </joint>
   <joint name="gimbal3" type="revolute">
-    <limit effort="1.5" velocity="6.0" lower="-3.14" upper="3.14"/>
+    <limit effort="1.5" velocity="6.0" lower="-1.0" upper="1.0"/>
     <parent link="main_body"/>
     <child link="gimbal3_link"/>
@@ -249,5 +249,5 @@
   </joint>
   <joint name="gimbal4" type="revolute">
-    <limit effort="1.5" velocity="6.0" lower="-3.14" upper="3.14"/>
+    <limit effort="1.5" velocity="6.0" lower="-1.0" upper="1.0"/>
     <parent link="main_body"/>
     <child link="gimbal4_link"/>
