Commit message: [gimbalrotor][grape] comment in visual mesh

File: robots/gimbalrotor/urdf/grape/gimbalrotor.urdf.xacro (robot description, xacro)
@@ -7,11 +7,11 @@
       <inertia ixx="0.0016139879539522" ixy="-5.366768549397e-07" ixz="-5.95600212021384e-07" iyy="0.00160428977142187" iyz="9.13377581199397e-08" izz="0.00305929998385753"/>
     </inertial>
-    <!-- <visual> -->
-    <!--   <geometry> -->
-    <!--     <mesh filename="package://gimbalrotor/urdf/grape/meshes/main_body.dae"/> -->
-    <!--   </geometry> -->
-    <!--   <material name="__unnamed_material_1"/> -->
-    <!--   <origin xyz="0.0 0.0 0.0" rpy="0.0 -0.0 0.0"/> -->
-    <!-- </visual> -->
+    <visual>
+      <geometry>
+        <mesh filename="package://gimbalrotor/urdf/grape/meshes/main_body.dae"/>
+      </geometry>
+      <material name="__unnamed_material_1"/>
+      <origin xyz="0.0 0.0 0.0" rpy="0.0 -0.0 0.0"/>
+    </visual>
     <!-- <collision> -->
     <!--   <geometry> -->
@@ -32,11 +32,11 @@
       <inertia ixx="6.23139432038947e-05" ixy="-6.80218913011022e-09" ixz="-2.71244742730139e-06" iyy="6.42832899579805e-05" iyz="-5.73083772407336e-09" izz="6.89107151163971e-05"/>
     </inertial>
-    <!-- <visual> -->
-    <!--   <geometry> -->
-    <!--     <mesh filename="package://gimbalrotor/urdf/grape/meshes/gimbal1_link.dae"/> -->
-    <!--   </geometry> -->
-    <!--   <material name="__unnamed_material_2"/> -->
-    <!--   <origin xyz="0.0 0.0 0.0" rpy="0.0 -0.0 0.0"/> -->
-    <!-- </visual> -->
+    <visual>
+      <geometry>
+        <mesh filename="package://gimbalrotor/urdf/grape/meshes/gimbal1_link.dae"/>
+      </geometry>
+      <material name="__unnamed_material_2"/>
+      <origin xyz="0.0 0.0 0.0" rpy="0.0 -0.0 0.0"/>
+    </visual>
     <!-- <collision> -->
     <!--   <geometry> -->
@@ -72,11 +72,11 @@
       <inertia ixx="6.23139432038948e-05" ixy="-6.80218913009929e-09" ixz="-2.7124474273014e-06" iyy="6.42832899579805e-05" iyz="-5.73083772406979e-09" izz="6.89107151163972e-05"/>
     </inertial>
-    <!-- <visual> -->
-    <!--   <geometry> -->
-    <!--     <mesh filename="package://gimbalrotor/urdf/grape/meshes/gimbal2_link.dae"/> -->
-    <!--   </geometry> -->
-    <!--   <material name="__unnamed_material_4"/> -->
-    <!--   <origin xyz="0.0 0.0 0.0" rpy="0.0 -0.0 0.0"/> -->
-    <!-- </visual> -->
+    <visual>
+      <geometry>
+        <mesh filename="package://gimbalrotor/urdf/grape/meshes/gimbal2_link.dae"/>
+      </geometry>
+      <material name="__unnamed_material_4"/>
+      <origin xyz="0.0 0.0 0.0" rpy="0.0 -0.0 0.0"/>
+    </visual>
     <!-- <collision> -->
     <!--   <geometry> -->
@@ -112,11 +112,11 @@
       <inertia ixx="6.23139432038948e-05" ixy="-6.80218913009913e-09" ixz="-2.71244742730139e-06" iyy="6.42832899579805e-05" iyz="-5.73083772407073e-09" izz="6.89107151163971e-05"/>
     </inertial>
-    <!-- <visual> -->
-    <!--   <geometry> -->
-    <!--     <mesh filename="package://gimbalrotor/urdf/grape/meshes/gimbal3_link.dae"/> -->
-    <!--   </geometry> -->
-    <!--   <material name="__unnamed_material_6"/> -->
-    <!--   <origin xyz="0.0 0.0 0.0" rpy="0.0 -0.0 0.0"/> -->
-    <!-- </visual> -->
+    <visual>
+      <geometry>
+        <mesh filename="package://gimbalrotor/urdf/grape/meshes/gimbal3_link.dae"/>
+      </geometry>
+      <material name="__unnamed_material_6"/>
+      <origin xyz="0.0 0.0 0.0" rpy="0.0 -0.0 0.0"/>
+    </visual>
     <!-- <collision> -->
     <!--   <geometry> -->
@@ -152,11 +152,11 @@
       <inertia ixx="6.23139432038948e-05" ixy="-6.80218913011076e-09" ixz="-2.7124474273014e-06" iyy="6.42832899579806e-05" iyz="-5.73083772407164e-09" izz="6.89107151163971e-05"/>
     </inertial>
-    <!-- <visual> -->
-    <!--   <geometry> -->
-    <!--     <mesh filename="package://gimbalrotor/urdf/grape/meshes/gimbal4_link.dae"/> -->
-    <!--   </geometry> -->
-    <!--   <material name="__unnamed_material_8"/> -->
-    <!--   <origin xyz="0.0 0.0 0.0" rpy="0.0 -0.0 0.0"/> -->
-    <!-- </visual> -->
+    <visual>
+      <geometry>
+        <mesh filename="package://gimbalrotor/urdf/grape/meshes/gimbal4_link.dae"/>
+      </geometry>
+      <material name="__unnamed_material_8"/>
+      <origin xyz="0.0 0.0 0.0" rpy="0.0 -0.0 0.0"/>
+    </visual>
     <!-- <collision> -->
     <!--   <geometry> -->
