Commit message: [gimbalrotor][grape] Fixed gazebo parameter

File: robots/gimbalrotor/robots/grape/gimbalrotor.urdf.xacro (robot description, xacro)
@@ -2,5 +2,5 @@
 <robot
     xmlns:xacro="http://www.ros.org/wiki/xacro" name="gimbalrotor" >
-    <xacro:include filename="$(find gimbalrotor)/urdf/grape/gimbalrotor.urdf.xacro" />
+    <xacro:include filename="$(find gimbalrotor)/urdf/grape/gimbalrotor_with_arm.urdf.xacro" />
     <xacro:include filename="$(find gimbalrotor)/urdf/grape/common.xacro" />
 </robot>

File: robots/gimbalrotor/urdf/grape/gimbalrotor_with_arm.urdf.xacro (robot description, xacro)
@@ -1,4 +1,4 @@
 <?xml version='1.0' encoding='UTF-8'?>
-<robot name="gimbalrotor_with_arm" xmlns:xacro="http://www.ros.org/wiki/xacro">
+<robot name="gimbalrotor" xmlns:xacro="http://www.ros.org/wiki/xacro">
   <xacro:include filename="$(find gimbalrotor)/urdf/grape/common.xacro"/>
   <xacro:include filename="$(find gimbalrotor)/urdf/grape/xacro/arm.xacro"/>

File: robots/gimbalrotor/urdf/grape/xacro/arm.xacro (robot description, xacro)
@@ -63,4 +63,55 @@
       xyz="0 0 0"
       rpy="0 0 0"/>
+    <!-- Transmissions for arm joints (required for Gazebo control) -->
+    <transmission name="arm_joint1_tran">
+      <type>transmission_interface/SimpleTransmission</type>
+      <joint name="arm_joint1_joint1">
+        <hardwareInterface>hardware_interface/EffortJointInterface</hardwareInterface>
+      </joint>
+      <actuator name="arm_servo1">
+        <hardwareInterface>hardware_interface/EffortJointInterface</hardwareInterface>
+        <mechanicalReduction>1</mechanicalReduction>
+      </actuator>
+    </transmission>
+    <transmission name="arm_joint2_tran">
+      <type>transmission_interface/SimpleTransmission</type>
+      <joint name="arm_joint2_joint1">
+        <hardwareInterface>hardware_interface/EffortJointInterface</hardwareInterface>
+      </joint>
+      <actuator name="arm_servo2">
+        <hardwareInterface>hardware_interface/EffortJointInterface</hardwareInterface>
+        <mechanicalReduction>1</mechanicalReduction>
+      </actuator>
+    </transmission>
+    <transmission name="arm_joint3_tran">
+      <type>transmission_interface/SimpleTransmission</type>
+      <joint name="arm_joint3_joint1">
+        <hardwareInterface>hardware_interface/EffortJointInterface</hardwareInterface>
+      </joint>
+      <actuator name="arm_servo3">
+        <hardwareInterface>hardware_interface/EffortJointInterface</hardwareInterface>
+        <mechanicalReduction>1</mechanicalReduction>
+      </actuator>
+    </transmission>
+    <transmission name="arm_joint4_tran">
+      <type>transmission_interface/SimpleTransmission</type>
+      <joint name="arm_joint4_joint1">
+        <hardwareInterface>hardware_interface/EffortJointInterface</hardwareInterface>
+      </joint>
+      <actuator name="arm_servo4">
+        <hardwareInterface>hardware_interface/EffortJointInterface</hardwareInterface>
+        <mechanicalReduction>1</mechanicalReduction>
+      </actuator>
+    </transmission>
+    <transmission name="arm_joint5_tran">
+      <type>transmission_interface/SimpleTransmission</type>
+      <joint name="arm_joint5_joint1">
+        <hardwareInterface>hardware_interface/EffortJointInterface</hardwareInterface>
+      </joint>
+      <actuator name="arm_servo5">
+        <hardwareInterface>hardware_interface/EffortJointInterface</hardwareInterface>
+        <mechanicalReduction>1</mechanicalReduction>
+      </actuator>
+    </transmission>
   </xacro:macro>
 </robot>
