Commit message: [gimbalrotor] change joint limit of screw_hinge_module_dynamixel

File: robots/gimbalrotor/urdf/grape/xacro/screw_hinge_module_dynamixel.xacro (robot description, xacro)
@@ -49,5 +49,6 @@
     <link name="${prefix}dummy_link"/>
     <joint name="${prefix}joint1" type="revolute">
-      <limit effort="0.0" velocity="0.0" lower="-0.567" upper="0.567"/>
+      <limit effort="0.0" velocity="0.0" lower="-3.141592" upper="3.141592"/>
+      <!-- <limit effort="0.0" velocity="0.0" lower="-0.567" upper="0.567"/> -->
       <parent link="${prefix}base_link"/>
       <child link="${prefix}link1"/>
