Commit message: change min thrust for bi-directional prop

File: robots/gimbalrotor/urdf/quad/common.xacro (robot description, xacro)
@@ -7,5 +7,5 @@
   <m_f_rate value="-0.0172" /> <!-- drug torque rate -->
   <xacro:property name="max_force" value="18.0" /> <!-- [N] -->
-  <xacro:property name="min_force" value="1.0" /> <!-- [N] -->
+  <xacro:property name="min_force" value="-10.0" /> <!-- [N] -->
   <!-- friction -->
   <xacro:macro name="friction" params="self">

File: robots/gimbalrotor/urdf/quad/gimbalrotor.urdf.xacro (robot description, xacro)
@@ -107,5 +107,5 @@
         <geometry>
           <box size="0.131 0.0325 0.065"/>
-        </geometry>p
+        </geometry>
       </collision>
     </link>

File: robots/mini_quadrotor/urdf/robot.urdf.xacro (robot description, xacro)
@@ -11,6 +11,6 @@
   <!-- dynamics -->
   <m_f_rate value="-0.011" /> <!-- drag torque rate -->
-  <xacro:property name="max_force" value="8.0" /> <!-- [N] -->
-  <xacro:property name="min_force" value="0.0" /> <!-- [N] -->
+  <xacro:property name="max_force" value="8.0" />  <!-- [N] -->
+  <xacro:property name="min_force" value="-8.0" /> <!-- [N] bidirectional -->
   <!-- friction -->
   <xacro:macro name="damping_factor" params="link">
