Commit message: add: collision definition and upper/lower/effort/velocity range, damping and friction

File: robots/hydragon/robots/robot.gazebo.xacro (robot description, xacro)
@@ -8,4 +8,40 @@
   <xacro:include filename="$(find aerial_robot_simulation)/xacro/spinal.gazebo.xacro" />
   <xacro:gazebo_spinal robot_name="$(arg robot_name)" />
+  <!-- friction -->
+  <xacro:macro name="friction" params="self">
+    <gazebo reference="front${self}_link">
+      <mu1>0.8</mu1>
+      <mu2>0.8</mu2>
+    </gazebo>
+    <gazebo reference="end${self}_link">
+      <mu1>0.8</mu1>
+      <mu2>0.8</mu2>
+    </gazebo>
+  </xacro:macro>
+  <xacro:macro name="damping_factor" params="link">
+    <gazebo reference="${link}">
+      <dampingFactor>0.00</dampingFactor>
+    </gazebo>
+  </xacro:macro>
+  <xacro:friction self="1"/>
+  <xacro:friction self="2"/>
+  <xacro:friction self="3"/>
+  <xacro:friction self="4"/>
+  <xacro:damping_factor link="front1_link"/>
+  <xacro:damping_factor link="front2_link"/>
+  <xacro:damping_factor link="front3_link"/>
+  <xacro:damping_factor link="front4_link"/>
+  <xacro:damping_factor link="end1_link"/>
+  <xacro:damping_factor link="end2_link"/>
+  <xacro:damping_factor link="end3_link"/>
+  <xacro:damping_factor link="end4_link"/>
+  <xacro:damping_factor link="gimbal1_link"/>
+  <xacro:damping_factor link="gimbal2_link"/>
+  <xacro:damping_factor link="gimbal3_link"/>
+  <xacro:damping_factor link="gimbal4_link"/>
+  <xacro:damping_factor link="duct1_link"/>
+  <xacro:damping_factor link="duct2_link"/>
+  <xacro:damping_factor link="duct3_link"/>
+  <xacro:damping_factor link="duct4_link"/>
   <gazebo reference="thrust1">
     <mu1>0.1</mu1>

File: robots/hydragon/urdf/common.xacro (robot description, xacro)
@@ -7,17 +7,22 @@
       <inertia ixx="0.00021055" ixy="3.1246e-10" ixz="-4.0813e-08" iyy="0.00010191" iyz="-4.0104e-07" izz="0.00021817"/>
     </inertial>
-    <!-- <visual> -->
-    <!--   <geometry> -->
-    <!--     <mesh filename="package://hydragon/meshes/front1_link.dae"/> -->
-    <!--   </geometry> -->
-    <!--   <material name="__unnamed_material_1"/> -->
-    <!--   <origin xyz="0.0 0.0 0.0" rpy="0.0 -0.0 0.0"/> -->
-    <!-- </visual> -->
-    <!-- <collision> -->
-    <!--   <geometry> -->
-    <!--     <mesh filename="package://hydragon/meshes/front1_link.stl"/> -->
-    <!--   </geometry> -->
-    <!--   <origin xyz="0.0 0.0 0.0" rpy="0.0 -0.0 0.0"/> -->
-    <!-- </collision> -->
+    <visual>
+      <geometry>
+        <mesh filename="package://hydragon/meshes/front1_link.stl"/>
+      </geometry>
+      <origin xyz="0.0 0.0 0.0" rpy="0.0 -0.0 0.0"/>
+    </visual>
+    <collision>
+      <geometry>
+        <box size="0.1025 0.02 0.02"/>
+      </geometry>
+      <origin xyz="-0.0707756 0 0" rpy="0 0 0"/>
+    </collision>
+    <collision>
+      <geometry>
+        <box size="0.034 0.0285 0.0465"/>
+      </geometry>
+      <origin xyz="-0.0710256 0 -0.039" rpy="0 0 0"/>
+    </collision>
   </link>
   <link name="body1_link">
@@ -27,17 +32,52 @@
       <inertia ixx="0.00016623" ixy="-3.3215e-07" ixz="-5.731e-09" iyy="0.00018621" iyz="-6.8029e-09" izz="0.00025293"/>
     </inertial>
-    <!-- <visual> -->
-    <!--   <geometry> -->
-    <!--     <mesh filename="package://hydragon/meshes/body1_link.dae"/> -->
-    <!--   </geometry> -->
-    <!--   <material name="__unnamed_material_2"/> -->
-    <!--   <origin xyz="0.0 0.0 0.0" rpy="0.0 -0.0 0.0"/> -->
-    <!-- </visual> -->
-    <!-- <collision> -->
-    <!--   <geometry> -->
-    <!--     <mesh filename="package://hydragon/meshes/body1_link.stl"/> -->
-    <!--   </geometry> -->
-    <!--   <origin xyz="0.0 0.0 0.0" rpy="0.0 -0.0 0.0"/> -->
-    <!-- </collision> -->
+    <visual>
+      <geometry>
+        <mesh filename="package://hydragon/meshes/body1_link.stl"/>
+      </geometry>
+      <origin xyz="0.0 0.0 0.0" rpy="0.0 -0.0 0.0"/>
+    </visual>
+    <collision>
+      <geometry>
+        <box size="0.133 0.010 0.030"/>
+      </geometry>
+      <origin xyz="-0.0459637 0.0796462 0" rpy="0 0 -1.0472"/>
+    </collision>
+    <collision>
+      <geometry>
+        <box size="0.133 0.010 0.030"/>
+      </geometry>
+      <origin xyz="-0.0459637 -0.0796462 0" rpy="0 0 1.0472"/>
+    </collision>
+    <collision>
+      <geometry>
+        <box size="0.166 0.010 0.030"/>
+      </geometry>
+      <origin xyz="-0.1699837 0.142 0" rpy="0 0 0"/>
+    </collision>
+    <collision>
+      <geometry>
+        <box size="0.166 0.010 0.030"/>
+      </geometry>
+      <origin xyz="-0.1699837 -0.142 0" rpy="0 0 0"/>
+    </collision>
+    <collision>
+      <geometry>
+        <box size="0.133 0.010 0.030"/>
+      </geometry>
+      <origin xyz="-0.2939837 0.0796462 0" rpy="0 0 1.0472"/>
+    </collision>
+    <collision>
+      <geometry>
+        <box size="0.133 0.010 0.030"/>
+      </geometry>
+      <origin xyz="-0.2939837 -0.0796462 0" rpy="0 0 -1.0472"/>
+    </collision>
+    <collision>
+      <geometry>
+        <box size="0.0465 0.034 0.0285"/>
+      </geometry>
+      <origin xyz="-0.1579837 0.166 0" rpy="0 0 0"/>
+    </collision>
   </link>
   <link name="duct1_link">
@@ -47,17 +87,10 @@
       <inertia ixx="0.0012194" ixy="2.2289e-07" ixz="-1.5989e-07" iyy="0.00099811" iyz="1.3306e-05" izz="0.0019906"/>
     </inertial>
-    <!-- <visual> -->
-    <!--   <geometry> -->
-    <!--     <mesh filename="package://hydragon/meshes/duct1_link.dae"/> -->
-    <!--   </geometry> -->
-    <!--   <material name="__unnamed_material_3"/> -->
-    <!--   <origin xyz="0.0 0.0 0.0" rpy="0.0 -0.0 0.0"/> -->
-    <!-- </visual> -->
-    <!-- <collision> -->
-    <!--   <geometry> -->
-    <!--     <mesh filename="package://hydragon/meshes/duct1_link.stl"/> -->
-    <!--   </geometry> -->
-    <!--   <origin xyz="0.0 0.0 0.0" rpy="0.0 -0.0 0.0"/> -->
-    <!-- </collision> -->
+    <visual>
+      <geometry>
+        <mesh filename="package://hydragon/meshes/duct1_link.stl"/>
+      </geometry>
+      <origin xyz="0.0 0.0 0.0" rpy="0.0 -0.0 0.0"/>
+    </visual>
   </link>
   <link name="thrust1">
@@ -69,7 +102,6 @@
     <visual>
       <geometry>
-        <mesh filename="package://hydragon/meshes/thrust1.dae"/>
-      </geometry>
-      <material name="__unnamed_material_4"/>
+        <mesh filename="package://hydragon/meshes/thrust1.stl"/>
+      </geometry>
       <origin xyz="0.0 0.0 0.0" rpy="0.0 -0.0 0.0"/>
     </visual>
@@ -88,17 +120,22 @@
       <inertia ixx="5.7571e-05" ixy="6.2131e-09" ixz="8.7034e-08" iyy="9.2786e-05" iyz="-8.9098e-12" izz="7.7319e-05"/>
     </inertial>
-    <!-- <visual> -->
-    <!--   <geometry> -->
-    <!--     <mesh filename="package://hydragon/meshes/end1_link.dae"/> -->
-    <!--   </geometry> -->
-    <!--   <material name="__unnamed_material_5"/> -->
-    <!--   <origin xyz="0.0 0.0 0.0" rpy="0.0 -0.0 0.0"/> -->
-    <!-- </visual> -->
-    <!-- <collision> -->
-    <!--   <geometry> -->
-    <!--     <mesh filename="package://hydragon/meshes/end1_link.stl"/> -->
-    <!--   </geometry> -->
-    <!--   <origin xyz="0.0 0.0 0.0" rpy="0.0 -0.0 0.0"/> -->
-    <!-- </collision> -->
+    <visual>
+      <geometry>
+        <mesh filename="package://hydragon/meshes/end1_link.stl"/>
+      </geometry>
+      <origin xyz="0.0 0.0 0.0" rpy="0.0 -0.0 0.0"/>
+    </visual>
+    <collision>
+      <geometry>
+        <box size="0.108 0.020 0.020"/>
+      </geometry>
+      <origin xyz="-0.0340163 0 0" rpy="0 0 0"/>
+    </collision>
+    <collision>
+      <geometry>
+        <box size="0.034 0.0285 0.0465"/>
+      </geometry>
+      <origin xyz="-0.0310163 0 -39" rpy="0 0 0"/>
+    </collision>
   </link>
   <link name="front2_link">
@@ -108,17 +145,22 @@
       <inertia ixx="0.00021055" ixy="3.1247e-10" ixz="-4.0813e-08" iyy="0.00010191" iyz="-4.0104e-07" izz="0.00021817"/>
     </inertial>
-    <!-- <visual> -->
-    <!--   <geometry> -->
-    <!--     <mesh filename="package://hydragon/meshes/front2_link.dae"/> -->
-    <!--   </geometry> -->
-    <!--   <material name="__unnamed_material_6"/> -->
-    <!--   <origin xyz="0.0 0.0 0.0" rpy="0.0 -0.0 0.0"/> -->
-    <!-- </visual> -->
-    <!-- <collision> -->
-    <!--   <geometry> -->
-    <!--     <mesh filename="package://hydragon/meshes/front2_link.stl"/> -->
-    <!--   </geometry> -->
-    <!--   <origin xyz="0.0 0.0 0.0" rpy="0.0 -0.0 0.0"/> -->
-    <!-- </collision> -->
+    <visual>
+      <geometry>
+        <mesh filename="package://hydragon/meshes/front2_link.stl"/>
+      </geometry>
+      <origin xyz="0.0 0.0 0.0" rpy="0.0 -0.0 0.0"/>
+    </visual>
+    <collision>
+      <geometry>
+        <box size="0.1025 0.02 0.02"/>
+      </geometry>
+      <origin xyz="-0.0707756 0 0" rpy="0 0 0"/>
+    </collision>
+    <collision>
+      <geometry>
+        <box size="0.034 0.0285 0.0465"/>
+      </geometry>
+      <origin xyz="-0.0710256 0 -0.039" rpy="0 0 0"/>
+    </collision>
   </link>
   <link name="body2_link">
@@ -128,17 +170,52 @@
       <inertia ixx="0.00016623" ixy="-3.3215e-07" ixz="-5.731e-09" iyy="0.00018621" iyz="-6.8029e-09" izz="0.00025293"/>
     </inertial>
-    <!-- <visual> -->
-    <!--   <geometry> -->
-    <!--     <mesh filename="package://hydragon/meshes/body2_link.dae"/> -->
-    <!--   </geometry> -->
-    <!--   <material name="__unnamed_material_7"/> -->
-    <!--   <origin xyz="0.0 0.0 0.0" rpy="0.0 -0.0 0.0"/> -->
-    <!-- </visual> -->
-    <!-- <collision> -->
-    <!--   <geometry> -->
-    <!--     <mesh filename="package://hydragon/meshes/body2_link.stl"/> -->
-    <!--   </geometry> -->
-    <!--   <origin xyz="0.0 0.0 0.0" rpy="0.0 -0.0 0.0"/> -->
-    <!-- </collision> -->
+    <visual>
+      <geometry>
+        <mesh filename="package://hydragon/meshes/body2_link.stl"/>
+      </geometry>
+      <origin xyz="0.0 0.0 0.0" rpy="0.0 -0.0 0.0"/>
+    </visual>
+    <collision>
+      <geometry>
+        <box size="0.133 0.010 0.030"/>
+      </geometry>
+      <origin xyz="-0.0459637 0.0796462 0" rpy="0 0 -1.0472"/>
+    </collision>
+    <collision>
+      <geometry>
+        <box size="0.133 0.010 0.030"/>
+      </geometry>
+      <origin xyz="-0.0459637 -0.0796462 0" rpy="0 0 1.0472"/>
+    </collision>
+    <collision>
+      <geometry>
+        <box size="0.166 0.010 0.030"/>
+      </geometry>
+      <origin xyz="-0.1699837 0.142 0" rpy="0 0 0"/>
+    </collision>
+    <collision>
+      <geometry>
+        <box size="0.166 0.010 0.030"/>
+      </geometry>
+      <origin xyz="-0.1699837 -0.142 0" rpy="0 0 0"/>
+    </collision>
+    <collision>
+      <geometry>
+        <box size="0.133 0.010 0.030"/>
+      </geometry>
+      <origin xyz="-0.2939837 0.0796462 0" rpy="0 0 1.0472"/>
+    </collision>
+    <collision>
+      <geometry>
+        <box size="0.133 0.010 0.030"/>
+      </geometry>
+      <origin xyz="-0.2939837 -0.0796462 0" rpy="0 0 -1.0472"/>
+    </collision>
+    <collision>
+      <geometry>
+        <box size="0.0465 0.034 0.0285"/>
+      </geometry>
+      <origin xyz="-0.1579837 0.166 0" rpy="0 0 0"/>
+    </collision>
   </link>
   <link name="duct2_link">
@@ -148,17 +225,10 @@
       <inertia ixx="0.0012194" ixy="2.2289e-07" ixz="-1.5989e-07" iyy="0.00099811" iyz="1.3306e-05" izz="0.0019906"/>
     </inertial>
-    <!-- <visual> -->
-    <!--   <geometry> -->
-    <!--     <mesh filename="package://hydragon/meshes/duct2_link.dae"/> -->
-    <!--   </geometry> -->
-    <!--   <material name="__unnamed_material_8"/> -->
-    <!--   <origin xyz="0.0 0.0 0.0" rpy="0.0 -0.0 0.0"/> -->
-    <!-- </visual> -->
-    <!-- <collision> -->
-    <!--   <geometry> -->
-    <!--     <mesh filename="package://hydragon/meshes/duct2_link.stl"/> -->
-    <!--   </geometry> -->
-    <!--   <origin xyz="0.0 0.0 0.0" rpy="0.0 -0.0 0.0"/> -->
-    <!-- </collision> -->
+    <visual>
+      <geometry>
+        <mesh filename="package://hydragon/meshes/duct2_link.stl"/>
+      </geometry>
+      <origin xyz="0.0 0.0 0.0" rpy="0.0 -0.0 0.0"/>
+    </visual>
   </link>
   <link name="thrust2">
@@ -170,7 +240,6 @@
     <visual>
       <geometry>
-        <mesh filename="package://hydragon/meshes/thrust2.dae"/>
-      </geometry>
-      <material name="__unnamed_material_9"/>
+        <mesh filename="package://hydragon/meshes/thrust2.stl"/>
+      </geometry>
       <origin xyz="0.0 0.0 0.0" rpy="0.0 -0.0 0.0"/>
     </visual>
@@ -189,17 +258,22 @@
       <inertia ixx="5.7571e-05" ixy="6.2131e-09" ixz="8.7034e-08" iyy="9.2786e-05" iyz="-8.9132e-12" izz="7.7319e-05"/>
     </inertial>
-    <!-- <visual> -->
-    <!--   <geometry> -->
-    <!--     <mesh filename="package://hydragon/meshes/end2_link.dae"/> -->
-    <!--   </geometry> -->
-    <!--   <material name="__unnamed_material_10"/> -->
-    <!--   <origin xyz="0.0 0.0 0.0" rpy="0.0 -0.0 0.0"/> -->
-    <!-- </visual> -->
-    <!-- <collision> -->
-    <!--   <geometry> -->
-    <!--     <mesh filename="package://hydragon/meshes/end2_link.stl"/> -->
-    <!--   </geometry> -->
-    <!--   <origin xyz="0.0 0.0 0.0" rpy="0.0 -0.0 0.0"/> -->
-    <!-- </collision> -->
+    <visual>
+      <geometry>
+        <mesh filename="package://hydragon/meshes/end2_link.stl"/>
+      </geometry>
+      <origin xyz="0.0 0.0 0.0" rpy="0.0 -0.0 0.0"/>
+    </visual>
+    <collision>
+      <geometry>
+        <box size="0.108 0.020 0.020"/>
+      </geometry>
+      <origin xyz="-0.0340163 0 0" rpy="0 0 0"/>
+    </collision>
+    <collision>
+      <geometry>
+        <box size="0.034 0.0285 0.0465"/>
+      </geometry>
+      <origin xyz="-0.0310163 0 -39" rpy="0 0 0"/>
+    </collision>
   </link>
   <link name="front3_link">
@@ -209,17 +283,22 @@
       <inertia ixx="0.00021055" ixy="3.1248e-10" ixz="-4.0813e-08" iyy="0.00010191" iyz="-4.0104e-07" izz="0.00021817"/>
     </inertial>
-    <!-- <visual> -->
-    <!--   <geometry> -->
-    <!--     <mesh filename="package://hydragon/meshes/front3_link.dae"/> -->
-    <!--   </geometry> -->
-    <!--   <material name="__unnamed_material_11"/> -->
-    <!--   <origin xyz="0.0 0.0 0.0" rpy="0.0 -0.0 0.0"/> -->
-    <!-- </visual> -->
-    <!-- <collision> -->
-    <!--   <geometry> -->
-    <!--     <mesh filename="package://hydragon/meshes/front3_link.stl"/> -->
-    <!--   </geometry> -->
-    <!--   <origin xyz="0.0 0.0 0.0" rpy="0.0 -0.0 0.0"/> -->
-    <!-- </collision> -->
+    <visual>
+      <geometry>
+        <mesh filename="package://hydragon/meshes/front3_link.stl"/>
+      </geometry>
+      <origin xyz="0.0 0.0 0.0" rpy="0.0 -0.0 0.0"/>
+    </visual>
+    <collision>
+      <geometry>
+        <box size="0.1025 0.02 0.02"/>
+      </geometry>
+      <origin xyz="-0.0707756 0 0" rpy="0 0 0"/>
+    </collision>
+    <collision>
+      <geometry>
+        <box size="0.034 0.0285 0.0465"/>
+      </geometry>
+      <origin xyz="-0.0710256 0 -0.039" rpy="0 0 0"/>
+    </collision>
   </link>
   <link name="body3_link">
@@ -229,17 +308,52 @@
       <inertia ixx="0.00016623" ixy="-3.3215e-07" ixz="-5.731e-09" iyy="0.00018621" iyz="-6.8029e-09" izz="0.00025293"/>
     </inertial>
-    <!-- <visual> -->
-    <!--   <geometry> -->
-    <!--     <mesh filename="package://hydragon/meshes/body3_link.dae"/> -->
-    <!--   </geometry> -->
-    <!--   <material name="__unnamed_material_12"/> -->
-    <!--   <origin xyz="0.0 0.0 0.0" rpy="0.0 -0.0 0.0"/> -->
-    <!-- </visual> -->
-    <!-- <collision> -->
-    <!--   <geometry> -->
-    <!--     <mesh filename="package://hydragon/meshes/body3_link.stl"/> -->
-    <!--   </geometry> -->
-    <!--   <origin xyz="0.0 0.0 0.0" rpy="0.0 -0.0 0.0"/> -->
-    <!-- </collision> -->
+    <visual>
+      <geometry>
+        <mesh filename="package://hydragon/meshes/body3_link.stl"/>
+      </geometry>
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