Commit message: [hydragon] temporaly comment out visual meshes

File: robots/hydragon/urdf/common.xacro (robot description, xacro)
@@ -7,11 +7,11 @@
       <inertia ixx="0.00021055" ixy="3.1246e-10" ixz="-4.0813e-08" iyy="0.00010191" iyz="-4.0104e-07" izz="0.00021817"/>
     </inertial>
-    <visual>
-      <geometry>
-        <mesh filename="package://hydragon/meshes/front1_link.dae"/>
-      </geometry>
-      <material name="__unnamed_material_1"/>
-      <origin xyz="0.0 0.0 0.0" rpy="0.0 -0.0 0.0"/>
-    </visual>
+    <!-- <visual> -->
+    <!--   <geometry> -->
+    <!--     <mesh filename="package://hydragon/meshes/front1_link.dae"/> -->
+    <!--   </geometry> -->
+    <!--   <material name="__unnamed_material_1"/> -->
+    <!--   <origin xyz="0.0 0.0 0.0" rpy="0.0 -0.0 0.0"/> -->
+    <!-- </visual> -->
     <!-- <collision> -->
     <!--   <geometry> -->
@@ -27,11 +27,11 @@
       <inertia ixx="0.00016623" ixy="-3.3215e-07" ixz="-5.731e-09" iyy="0.00018621" iyz="-6.8029e-09" izz="0.00025293"/>
     </inertial>
-    <visual>
-      <geometry>
-        <mesh filename="package://hydragon/meshes/body1_link.dae"/>
-      </geometry>
-      <material name="__unnamed_material_2"/>
-      <origin xyz="0.0 0.0 0.0" rpy="0.0 -0.0 0.0"/>
-    </visual>
+    <!-- <visual> -->
+    <!--   <geometry> -->
+    <!--     <mesh filename="package://hydragon/meshes/body1_link.dae"/> -->
+    <!--   </geometry> -->
+    <!--   <material name="__unnamed_material_2"/> -->
+    <!--   <origin xyz="0.0 0.0 0.0" rpy="0.0 -0.0 0.0"/> -->
+    <!-- </visual> -->
     <!-- <collision> -->
     <!--   <geometry> -->
@@ -47,11 +47,11 @@
       <inertia ixx="0.0012194" ixy="2.2289e-07" ixz="-1.5989e-07" iyy="0.00099811" iyz="1.3306e-05" izz="0.0019906"/>
     </inertial>
-    <visual>
-      <geometry>
-        <mesh filename="package://hydragon/meshes/duct1_link.dae"/>
-      </geometry>
-      <material name="__unnamed_material_3"/>
-      <origin xyz="0.0 0.0 0.0" rpy="0.0 -0.0 0.0"/>
-    </visual>
+    <!-- <visual> -->
+    <!--   <geometry> -->
+    <!--     <mesh filename="package://hydragon/meshes/duct1_link.dae"/> -->
+    <!--   </geometry> -->
+    <!--   <material name="__unnamed_material_3"/> -->
+    <!--   <origin xyz="0.0 0.0 0.0" rpy="0.0 -0.0 0.0"/> -->
+    <!-- </visual> -->
     <!-- <collision> -->
     <!--   <geometry> -->
@@ -74,10 +74,11 @@
       <origin xyz="0.0 0.0 0.0" rpy="0.0 -0.0 0.0"/>
     </visual>
-    <!-- <collision> -->
-    <!--   <geometry> -->
-    <!--     <mesh filename="package://hydragon/meshes/thrust1.stl"/> -->
-    <!--   </geometry> -->
-    <!--   <origin xyz="0.0 0.0 0.0" rpy="0.0 -0.0 0.0"/> -->
-    <!-- </collision> -->
+    <collision>
+      <geometry>
+        <!--     <mesh filename="package://hydragon/meshes/thrust1.stl"/> -->
+        <cylinder radius="0.125" length="0.1"/>
+      </geometry>
+      <origin xyz="0.0 0.0 0.0" rpy="0.0 -0.0 0.0"/>
+    </collision>
   </link>
   <link name="end1_link">
@@ -87,11 +88,11 @@
       <inertia ixx="5.7571e-05" ixy="6.2131e-09" ixz="8.7034e-08" iyy="9.2786e-05" iyz="-8.9098e-12" izz="7.7319e-05"/>
     </inertial>
-    <visual>
-      <geometry>
-        <mesh filename="package://hydragon/meshes/end1_link.dae"/>
-      </geometry>
-      <material name="__unnamed_material_5"/>
-      <origin xyz="0.0 0.0 0.0" rpy="0.0 -0.0 0.0"/>
-    </visual>
+    <!-- <visual> -->
+    <!--   <geometry> -->
+    <!--     <mesh filename="package://hydragon/meshes/end1_link.dae"/> -->
+    <!--   </geometry> -->
+    <!--   <material name="__unnamed_material_5"/> -->
+    <!--   <origin xyz="0.0 0.0 0.0" rpy="0.0 -0.0 0.0"/> -->
+    <!-- </visual> -->
     <!-- <collision> -->
     <!--   <geometry> -->
@@ -107,11 +108,11 @@
       <inertia ixx="0.00021055" ixy="3.1247e-10" ixz="-4.0813e-08" iyy="0.00010191" iyz="-4.0104e-07" izz="0.00021817"/>
     </inertial>
-    <visual>
-      <geometry>
-        <mesh filename="package://hydragon/meshes/front2_link.dae"/>
-      </geometry>
-      <material name="__unnamed_material_6"/>
-      <origin xyz="0.0 0.0 0.0" rpy="0.0 -0.0 0.0"/>
-    </visual>
+    <!-- <visual> -->
+    <!--   <geometry> -->
+    <!--     <mesh filename="package://hydragon/meshes/front2_link.dae"/> -->
+    <!--   </geometry> -->
+    <!--   <material name="__unnamed_material_6"/> -->
+    <!--   <origin xyz="0.0 0.0 0.0" rpy="0.0 -0.0 0.0"/> -->
+    <!-- </visual> -->
     <!-- <collision> -->
     <!--   <geometry> -->
@@ -127,11 +128,11 @@
       <inertia ixx="0.00016623" ixy="-3.3215e-07" ixz="-5.731e-09" iyy="0.00018621" iyz="-6.8029e-09" izz="0.00025293"/>
     </inertial>
-    <visual>
-      <geometry>
-        <mesh filename="package://hydragon/meshes/body2_link.dae"/>
-      </geometry>
-      <material name="__unnamed_material_7"/>
-      <origin xyz="0.0 0.0 0.0" rpy="0.0 -0.0 0.0"/>
-    </visual>
+    <!-- <visual> -->
+    <!--   <geometry> -->
+    <!--     <mesh filename="package://hydragon/meshes/body2_link.dae"/> -->
+    <!--   </geometry> -->
+    <!--   <material name="__unnamed_material_7"/> -->
+    <!--   <origin xyz="0.0 0.0 0.0" rpy="0.0 -0.0 0.0"/> -->
+    <!-- </visual> -->
     <!-- <collision> -->
     <!--   <geometry> -->
@@ -147,11 +148,11 @@
       <inertia ixx="0.0012194" ixy="2.2289e-07" ixz="-1.5989e-07" iyy="0.00099811" iyz="1.3306e-05" izz="0.0019906"/>
     </inertial>
-    <visual>
-      <geometry>
-        <mesh filename="package://hydragon/meshes/duct2_link.dae"/>
-      </geometry>
-      <material name="__unnamed_material_8"/>
-      <origin xyz="0.0 0.0 0.0" rpy="0.0 -0.0 0.0"/>
-    </visual>
+    <!-- <visual> -->
+    <!--   <geometry> -->
+    <!--     <mesh filename="package://hydragon/meshes/duct2_link.dae"/> -->
+    <!--   </geometry> -->
+    <!--   <material name="__unnamed_material_8"/> -->
+    <!--   <origin xyz="0.0 0.0 0.0" rpy="0.0 -0.0 0.0"/> -->
+    <!-- </visual> -->
     <!-- <collision> -->
     <!--   <geometry> -->
@@ -174,10 +175,11 @@
       <origin xyz="0.0 0.0 0.0" rpy="0.0 -0.0 0.0"/>
     </visual>
-    <!-- <collision> -->
-    <!--   <geometry> -->
-    <!--     <mesh filename="package://hydragon/meshes/thrust2.stl"/> -->
-    <!--   </geometry> -->
-    <!--   <origin xyz="0.0 0.0 0.0" rpy="0.0 -0.0 0.0"/> -->
-    <!-- </collision> -->
+    <collision>
+      <geometry>
+        <!--     <mesh filename="package://hydragon/meshes/thrust2.stl"/> -->
+        <cylinder radius="0.125" length="0.1"/>
+      </geometry>
+      <origin xyz="0.0 0.0 0.0" rpy="0.0 -0.0 0.0"/>
+    </collision>
   </link>
   <link name="end2_link">
@@ -187,11 +189,11 @@
       <inertia ixx="5.7571e-05" ixy="6.2131e-09" ixz="8.7034e-08" iyy="9.2786e-05" iyz="-8.9132e-12" izz="7.7319e-05"/>
     </inertial>
-    <visual>
-      <geometry>
-        <mesh filename="package://hydragon/meshes/end2_link.dae"/>
-      </geometry>
-      <material name="__unnamed_material_10"/>
-      <origin xyz="0.0 0.0 0.0" rpy="0.0 -0.0 0.0"/>
-    </visual>
+    <!-- <visual> -->
+    <!--   <geometry> -->
+    <!--     <mesh filename="package://hydragon/meshes/end2_link.dae"/> -->
+    <!--   </geometry> -->
+    <!--   <material name="__unnamed_material_10"/> -->
+    <!--   <origin xyz="0.0 0.0 0.0" rpy="0.0 -0.0 0.0"/> -->
+    <!-- </visual> -->
     <!-- <collision> -->
     <!--   <geometry> -->
@@ -207,11 +209,11 @@
       <inertia ixx="0.00021055" ixy="3.1248e-10" ixz="-4.0813e-08" iyy="0.00010191" iyz="-4.0104e-07" izz="0.00021817"/>
     </inertial>
-    <visual>
-      <geometry>
-        <mesh filename="package://hydragon/meshes/front3_link.dae"/>
-      </geometry>
-      <material name="__unnamed_material_11"/>
-      <origin xyz="0.0 0.0 0.0" rpy="0.0 -0.0 0.0"/>
-    </visual>
+    <!-- <visual> -->
+    <!--   <geometry> -->
+    <!--     <mesh filename="package://hydragon/meshes/front3_link.dae"/> -->
+    <!--   </geometry> -->
+    <!--   <material name="__unnamed_material_11"/> -->
+    <!--   <origin xyz="0.0 0.0 0.0" rpy="0.0 -0.0 0.0"/> -->
+    <!-- </visual> -->
     <!-- <collision> -->
     <!--   <geometry> -->
@@ -227,11 +229,11 @@
       <inertia ixx="0.00016623" ixy="-3.3215e-07" ixz="-5.731e-09" iyy="0.00018621" iyz="-6.8029e-09" izz="0.00025293"/>
     </inertial>
-    <visual>
-      <geometry>
-        <mesh filename="package://hydragon/meshes/body3_link.dae"/>
-      </geometry>
-      <material name="__unnamed_material_12"/>
-      <origin xyz="0.0 0.0 0.0" rpy="0.0 -0.0 0.0"/>
-    </visual>
+    <!-- <visual> -->
+    <!--   <geometry> -->
+    <!--     <mesh filename="package://hydragon/meshes/body3_link.dae"/> -->
+    <!--   </geometry> -->
+    <!--   <material name="__unnamed_material_12"/> -->
+    <!--   <origin xyz="0.0 0.0 0.0" rpy="0.0 -0.0 0.0"/> -->
+    <!-- </visual> -->
     <!-- <collision> -->
     <!--   <geometry> -->
@@ -247,11 +249,11 @@
       <inertia ixx="0.0012194" ixy="2.2289e-07" ixz="-1.5989e-07" iyy="0.00099811" iyz="1.3306e-05" izz="0.0019906"/>
     </inertial>
-    <visual>
-      <geometry>
-        <mesh filename="package://hydragon/meshes/duct3_link.dae"/>
-      </geometry>
-      <material name="__unnamed_material_13"/>
-      <origin xyz="0.0 0.0 0.0" rpy="0.0 -0.0 0.0"/>
-    </visual>
+    <!-- <visual> -->
+    <!--   <geometry> -->
+    <!--     <mesh filename="package://hydragon/meshes/duct3_link.dae"/> -->
+    <!--   </geometry> -->
+    <!--   <material name="__unnamed_material_13"/> -->
+    <!--   <origin xyz="0.0 0.0 0.0" rpy="0.0 -0.0 0.0"/> -->
+    <!-- </visual> -->
     <!-- <collision> -->
     <!--   <geometry> -->
@@ -274,10 +276,11 @@
       <origin xyz="0.0 0.0 0.0" rpy="0.0 -0.0 0.0"/>
     </visual>
-    <!-- <collision> -->
-    <!--   <geometry> -->
-    <!--     <mesh filename="package://hydragon/meshes/thrust3.stl"/> -->
-    <!--   </geometry> -->
-    <!--   <origin xyz="0.0 0.0 0.0" rpy="0.0 -0.0 0.0"/> -->
-    <!-- </collision> -->
+    <collision>
+      <geometry>
+        <!--     <mesh filename="package://hydragon/meshes/thrust3.stl"/> -->
+        <cylinder radius="0.125" length="0.1"/>
+      </geometry>
+      <origin xyz="0.0 0.0 0.0" rpy="0.0 -0.0 0.0"/>
+    </collision>
   </link>
   <link name="end3_link">
@@ -287,11 +290,11 @@
       <inertia ixx="5.7571e-05" ixy="6.2131e-09" ixz="8.7034e-08" iyy="9.2786e-05" iyz="-8.9132e-12" izz="7.7319e-05"/>
     </inertial>
-    <visual>
-      <geometry>
-        <mesh filename="package://hydragon/meshes/end3_link.dae"/>
-      </geometry>
-      <material name="__unnamed_material_15"/>
-      <origin xyz="0.0 0.0 0.0" rpy="0.0 -0.0 0.0"/>
-    </visual>
+    <!-- <visual> -->
+    <!--   <geometry> -->
+    <!--     <mesh filename="package://hydragon/meshes/end3_link.dae"/> -->
+    <!--   </geometry> -->
+    <!--   <material name="__unnamed_material_15"/> -->
+    <!--   <origin xyz="0.0 0.0 0.0" rpy="0.0 -0.0 0.0"/> -->
+    <!-- </visual> -->
     <!-- <collision> -->
     <!--   <geometry> -->
@@ -307,11 +310,11 @@
       <inertia ixx="0.00021055" ixy="3.1248e-10" ixz="-4.0813e-08" iyy="0.00010191" iyz="-4.0104e-07" izz="0.00021817"/>
     </inertial>
-    <visual>
-      <geometry>
-        <mesh filename="package://hydragon/meshes/front4_link.dae"/>
-      </geometry>
-      <material name="__unnamed_material_16"/>
-      <origin xyz="0.0 0.0 0.0" rpy="0.0 -0.0 0.0"/>
-    </visual>
+    <!-- <visual> -->
+    <!--   <geometry> -->
+    <!--     <mesh filename="package://hydragon/meshes/front4_link.dae"/> -->
+    <!--   </geometry> -->
+    <!--   <material name="__unnamed_material_16"/> -->
+    <!--   <origin xyz="0.0 0.0 0.0" rpy="0.0 -0.0 0.0"/> -->
+    <!-- </visual> -->
     <!-- <collision> -->
     <!--   <geometry> -->
@@ -327,11 +330,11 @@
       <inertia ixx="0.00016623" ixy="-3.3215e-07" ixz="-5.731e-09" iyy="0.00018621" iyz="-6.8029e-09" izz="0.00025293"/>
     </inertial>
-    <visual>
-      <geometry>
-        <mesh filename="package://hydragon/meshes/body4_link.dae"/>
-      </geometry>
-      <material name="__unnamed_material_17"/>
-      <origin xyz="0.0 0.0 0.0" rpy="0.0 -0.0 0.0"/>
-    </visual>
+    <!-- <visual> -->
+    <!--   <geometry> -->
+    <!--     <mesh filename="package://hydragon/meshes/body4_link.dae"/> -->
+    <!--   </geometry> -->
+    <!--   <material name="__unnamed_material_17"/> -->
+    <!--   <origin xyz="0.0 0.0 0.0" rpy="0.0 -0.0 0.0"/> -->
+    <!-- </visual> -->
     <!-- <collision> -->
     <!--   <geometry> -->
@@ -347,11 +350,11 @@
       <inertia ixx="0.0012194" ixy="2.2289e-07" ixz="-1.5989e-07" iyy="0.00099811" iyz="1.3306e-05" izz="0.0019906"/>
     </inertial>
-    <visual>
-      <geometry>
-        <mesh filename="package://hydragon/meshes/duct4_link.dae"/>
-      </geometry>
-      <material name="__unnamed_material_18"/>
-      <origin xyz="0.0 0.0 0.0" rpy="0.0 -0.0 0.0"/>
-    </visual>
+    <!-- <visual> -->
+    <!--   <geometry> -->
+    <!--     <mesh filename="package://hydragon/meshes/duct4_link.dae"/> -->
+    <!--   </geometry> -->
+    <!--   <material name="__unnamed_material_18"/> -->
+    <!--   <origin xyz="0.0 0.0 0.0" rpy="0.0 -0.0 0.0"/> -->
+    <!-- </visual> -->
     <!-- <collision> -->
     <!--   <geometry> -->
@@ -374,10 +377,11 @@
       <origin xyz="0.0 0.0 0.0" rpy="0.0 -0.0 0.0"/>
     </visual>
-    <!-- <collision> -->
-    <!--   <geometry> -->
-    <!--     <mesh filename="package://hydragon/meshes/thrust4.stl"/> -->
-    <!--   </geometry> -->
-    <!--   <origin xyz="0.0 0.0 0.0" rpy="0.0 -0.0 0.0"/> -->
-    <!-- </collision> -->
+    <collision>
+      <geometry>
+        <!--     <mesh filename="package://hydragon/meshes/thrust4.stl"/> -->
+        <cylinder radius="0.125" length="0.1"/>
+      </geometry>
+      <origin xyz="0.0 0.0 0.0" rpy="0.0 -0.0 0.0"/>
+    </collision>
   </link>
   <link name="end4_link">
@@ -387,11 +391,11 @@
       <inertia ixx="5.7571e-05" ixy="6.2131e-09" ixz="8.7034e-08" iyy="9.2786e-05" iyz="-8.9133e-12" izz="7.7319e-05"/>
     </inertial>
-    <visual>
-      <geometry>
-        <mesh filename="package://hydragon/meshes/end4_link.dae"/>
-      </geometry>
-      <material name="__unnamed_material_20"/>
-      <origin xyz="0.0 0.0 0.0" rpy="0.0 -0.0 0.0"/>
-    </visual>
+    <!-- <visual> -->
+    <!--   <geometry> -->
+    <!--     <mesh filename="package://hydragon/meshes/end4_link.dae"/> -->
+    <!--   </geometry> -->
+    <!--   <material name="__unnamed_material_20"/> -->
+    <!--   <origin xyz="0.0 0.0 0.0" rpy="0.0 -0.0 0.0"/> -->
+    <!-- </visual> -->
     <!-- <collision> -->
     <!--   <geometry> -->
@@ -407,11 +411,11 @@
       <inertia ixx="1.8175e-06" ixy="3.5211e-09" ixz="2.4144e-11" iyy="1.8131e-06" iyz="-1.8205e-10" izz="3.6133e-06"/>
     </inertial>
-    <visual>
-      <geometry>
-        <mesh filename="package://hydragon/meshes/fc.dae"/>
-      </geometry>
-      <material name="__unnamed_material_21"/>
-      <origin xyz="0.0 0.0 0.0" rpy="0.0 -0.0 0.0"/>
-    </visual>
+    <!-- <visual> -->
+    <!--   <geometry> -->
+    <!--     <mesh filename="package://hydragon/meshes/fc.dae"/> -->
+    <!--   </geometry> -->
+    <!--   <material name="__unnamed_material_21"/> -->
+    <!--   <origin xyz="0.0 0.0 0.0" rpy="0.0 -0.0 0.0"/> -->
+    <!-- </visual> -->
     <!-- <collision> -->
     <!--   <geometry> -->
