Commit message: [hydragon] fix collision to spawn in gazebo

File: robots/hydragon/urdf/common.xacro (robot description, xacro)
@@ -13,13 +13,13 @@
       <origin xyz="0.0 0.0 0.0" rpy="0.0 -0.0 0.0"/>
     </visual>
-    <collision>
-      <geometry>
-        <box size="0.1025 0.02 0.02"/>
-      </geometry>
-      <origin xyz="-0.0707756 0 0" rpy="0 0 0"/>
-    </collision>
-    <collision>
-      <geometry>
-        <box size="0.034 0.0285 0.0465"/>
+    <!-- <collision> -->
+    <!--   <geometry> -->
+    <!--     <box size="0.1025 0.02 0.02"/> -->
+    <!--   </geometry> -->
+    <!--   <origin xyz="-0.0707756 0 0" rpy="0 0 0"/> -->
+    <!-- </collision> -->
+    <collision>
+      <geometry>
+        <box size="0.1 0.1 0.2"/>
       </geometry>
       <origin xyz="-0.0710256 0 -0.039" rpy="0 0 0"/>
@@ -38,46 +38,44 @@
       <origin xyz="0.0 0.0 0.0" rpy="0.0 -0.0 0.0"/>
     </visual>
-    <collision>
-      <geometry>
-        <box size="0.133 0.010 0.030"/>
-      </geometry>
-      <origin xyz="-0.0459637 0.0796462 0" rpy="0 0 -1.0472"/>
-    </collision>
-    <collision>
-      <geometry>
-        <box size="0.133 0.010 0.030"/>
-      </geometry>
-      <origin xyz="-0.0459637 -0.0796462 0" rpy="0 0 1.0472"/>
-    </collision>
-    <collision>
-      <geometry>
-        <box size="0.166 0.010 0.030"/>
-      </geometry>
-      <origin xyz="-0.1699837 0.142 0" rpy="0 0 0"/>
-    </collision>
-    <collision>
-      <geometry>
-        <box size="0.166 0.010 0.030"/>
-      </geometry>
-      <origin xyz="-0.1699837 -0.142 0" rpy="0 0 0"/>
-    </collision>
-    <collision>
-      <geometry>
-        <box size="0.133 0.010 0.030"/>
-      </geometry>
-      <origin xyz="-0.2939837 0.0796462 0" rpy="0 0 1.0472"/>
-    </collision>
-    <collision>
-      <geometry>
-        <box size="0.133 0.010 0.030"/>
-      </geometry>
-      <origin xyz="-0.2939837 -0.0796462 0" rpy="0 0 -1.0472"/>
-    </collision>
-    <collision>
-      <geometry>
-        <box size="0.0465 0.034 0.0285"/>
-      </geometry>
-      <origin xyz="-0.1579837 0.166 0" rpy="0 0 0"/>
-    </collision>
+    <!--     <box size="0.133 0.010 0.030"/> -->
+    <!--   </geometry> -->
+    <!--   <origin xyz="-0.0459637 0.0796462 0" rpy="0 0 -1.0472"/> -->
+    <!-- </collision> -->
+    <!-- <collision> -->
+    <!--   <geometry> -->
+    <!--     <box size="0.133 0.010 0.030"/> -->
+    <!--   </geometry> -->
+    <!--   <origin xyz="-0.0459637 -0.0796462 0" rpy="0 0 1.0472"/> -->
+    <!-- </collision> -->
+    <!-- <collision> -->
+    <!--   <geometry> -->
+    <!--     <box size="0.166 0.010 0.030"/> -->
+    <!--   </geometry> -->
+    <!--   <origin xyz="-0.1699837 0.142 0" rpy="0 0 0"/> -->
+    <!-- </collision> -->
+    <!-- <collision> -->
+    <!--   <geometry> -->
+    <!--     <box size="0.166 0.010 0.030"/> -->
+    <!--   </geometry> -->
+    <!--   <origin xyz="-0.1699837 -0.142 0" rpy="0 0 0"/> -->
+    <!-- </collision> -->
+    <!-- <collision> -->
+    <!--   <geometry> -->
+    <!--     <box size="0.133 0.010 0.030"/> -->
+    <!--   </geometry> -->
+    <!--   <origin xyz="-0.2939837 0.0796462 0" rpy="0 0 1.0472"/> -->
+    <!-- </collision> -->
+    <!-- <collision> -->
+    <!--   <geometry> -->
+    <!--     <box size="0.133 0.010 0.030"/> -->
+    <!--   </geometry> -->
+    <!--   <origin xyz="-0.2939837 -0.0796462 0" rpy="0 0 -1.0472"/> -->
+    <!-- </collision> -->
+    <!-- <collision> -->
+    <!--   <geometry> -->
+    <!--     <box size="0.0465 0.034 0.0285"/> -->
+    <!--   </geometry> -->
+    <!--   <origin xyz="-0.1579837 0.166 0" rpy="0 0 0"/> -->
+    <!-- </collision> -->
   </link>
   <link name="duct1_link">
@@ -128,14 +126,14 @@
     <collision>
       <geometry>
-        <box size="0.108 0.020 0.020"/>
-      </geometry>
-      <origin xyz="-0.0340163 0 0" rpy="0 0 0"/>
-    </collision>
-    <collision>
-      <geometry>
-        <box size="0.034 0.0285 0.0465"/>
-      </geometry>
-      <origin xyz="-0.0310163 0 -39" rpy="0 0 0"/>
-    </collision>
+        <box size="0.1 0.1 0.2"/>
+      </geometry>
+      <origin xyz="-0.0340163 0 -0.039" rpy="0 0 0"/>
+    </collision>
+    <!-- <collision> -->
+    <!--   <geometry> -->
+    <!--     <box size="0.034 0.0285 0.0465"/> -->
+    <!--   </geometry> -->
+    <!--   <origin xyz="-0.0310163 0 -39" rpy="0 0 0"/> -->
+    <!-- </collision> -->
   </link>
   <link name="front2_link">
@@ -151,13 +149,13 @@
       <origin xyz="0.0 0.0 0.0" rpy="0.0 -0.0 0.0"/>
     </visual>
-    <collision>
-      <geometry>
-        <box size="0.1025 0.02 0.02"/>
-      </geometry>
-      <origin xyz="-0.0707756 0 0" rpy="0 0 0"/>
-    </collision>
-    <collision>
-      <geometry>
-        <box size="0.034 0.0285 0.0465"/>
+    <!-- <collision> -->
+    <!--   <geometry> -->
+    <!--     <box size="0.1025 0.02 0.02"/> -->
+    <!--   </geometry> -->
+    <!--   <origin xyz="-0.0707756 0 0" rpy="0 0 0"/> -->
+    <!-- </collision> -->
+    <collision>
+      <geometry>
+        <box size="0.1 0.1 0.2"/>
       </geometry>
       <origin xyz="-0.0710256 0 -0.039" rpy="0 0 0"/>
@@ -176,46 +174,46 @@
       <origin xyz="0.0 0.0 0.0" rpy="0.0 -0.0 0.0"/>
     </visual>
-    <collision>
-      <geometry>
-        <box size="0.133 0.010 0.030"/>
-      </geometry>
-      <origin xyz="-0.0459637 0.0796462 0" rpy="0 0 -1.0472"/>
-    </collision>
-    <collision>
-      <geometry>
-        <box size="0.133 0.010 0.030"/>
-      </geometry>
-      <origin xyz="-0.0459637 -0.0796462 0" rpy="0 0 1.0472"/>
-    </collision>
-    <collision>
-      <geometry>
-        <box size="0.166 0.010 0.030"/>
-      </geometry>
-      <origin xyz="-0.1699837 0.142 0" rpy="0 0 0"/>
-    </collision>
-    <collision>
-      <geometry>
-        <box size="0.166 0.010 0.030"/>
-      </geometry>
-      <origin xyz="-0.1699837 -0.142 0" rpy="0 0 0"/>
-    </collision>
-    <collision>
-      <geometry>
-        <box size="0.133 0.010 0.030"/>
-      </geometry>
-      <origin xyz="-0.2939837 0.0796462 0" rpy="0 0 1.0472"/>
-    </collision>
-    <collision>
-      <geometry>
-        <box size="0.133 0.010 0.030"/>
-      </geometry>
-      <origin xyz="-0.2939837 -0.0796462 0" rpy="0 0 -1.0472"/>
-    </collision>
-    <collision>
-      <geometry>
-        <box size="0.0465 0.034 0.0285"/>
-      </geometry>
-      <origin xyz="-0.1579837 0.166 0" rpy="0 0 0"/>
-    </collision>
+    <!-- <collision> -->
+    <!--   <geometry> -->
+    <!--     <box size="0.133 0.010 0.030"/> -->
+    <!--   </geometry> -->
+    <!--   <origin xyz="-0.0459637 0.0796462 0" rpy="0 0 -1.0472"/> -->
+    <!-- </collision> -->
+    <!-- <collision> -->
+    <!--   <geometry> -->
+    <!--     <box size="0.133 0.010 0.030"/> -->
+    <!--   </geometry> -->
+    <!--   <origin xyz="-0.0459637 -0.0796462 0" rpy="0 0 1.0472"/> -->
+    <!-- </collision> -->
+    <!-- <collision> -->
+    <!--   <geometry> -->
+    <!--     <box size="0.166 0.010 0.030"/> -->
+    <!--   </geometry> -->
+    <!--   <origin xyz="-0.1699837 0.142 0" rpy="0 0 0"/> -->
+    <!-- </collision> -->
+    <!-- <collision> -->
+    <!--   <geometry> -->
+    <!--     <box size="0.166 0.010 0.030"/> -->
+    <!--   </geometry> -->
+    <!--   <origin xyz="-0.1699837 -0.142 0" rpy="0 0 0"/> -->
+    <!-- </collision> -->
+    <!-- <collision> -->
+    <!--   <geometry> -->
+    <!--     <box size="0.133 0.010 0.030"/> -->
+    <!--   </geometry> -->
+    <!--   <origin xyz="-0.2939837 0.0796462 0" rpy="0 0 1.0472"/> -->
+    <!-- </collision> -->
+    <!-- <collision> -->
+    <!--   <geometry> -->
+    <!--     <box size="0.133 0.010 0.030"/> -->
+    <!--   </geometry> -->
+    <!--   <origin xyz="-0.2939837 -0.0796462 0" rpy="0 0 -1.0472"/> -->
+    <!-- </collision> -->
+    <!-- <collision> -->
+    <!--   <geometry> -->
+    <!--     <box size="0.0465 0.034 0.0285"/> -->
+    <!--   </geometry> -->
+    <!--   <origin xyz="-0.1579837 0.166 0" rpy="0 0 0"/> -->
+    <!-- </collision> -->
   </link>
   <link name="duct2_link">
@@ -266,14 +264,14 @@
     <collision>
       <geometry>
-        <box size="0.108 0.020 0.020"/>
-      </geometry>
-      <origin xyz="-0.0340163 0 0" rpy="0 0 0"/>
-    </collision>
-    <collision>
-      <geometry>
-        <box size="0.034 0.0285 0.0465"/>
-      </geometry>
-      <origin xyz="-0.0310163 0 -39" rpy="0 0 0"/>
-    </collision>
+        <box size="0.1 0.1 0.2"/>
+      </geometry>
+      <origin xyz="-0.0340163 0 -0.039" rpy="0 0 0"/>
+    </collision>
+    <!-- <collision> -->
+    <!--   <geometry> -->
+    <!--     <box size="0.034 0.0285 0.0465"/> -->
+    <!--   </geometry> -->
+    <!--   <origin xyz="-0.0310163 0 -39" rpy="0 0 0"/> -->
+    <!-- </collision> -->
   </link>
   <link name="front3_link">
@@ -289,13 +287,13 @@
       <origin xyz="0.0 0.0 0.0" rpy="0.0 -0.0 0.0"/>
     </visual>
-    <collision>
-      <geometry>
-        <box size="0.1025 0.02 0.02"/>
-      </geometry>
-      <origin xyz="-0.0707756 0 0" rpy="0 0 0"/>
-    </collision>
-    <collision>
-      <geometry>
-        <box size="0.034 0.0285 0.0465"/>
+    <!-- <collision> -->
+    <!--   <geometry> -->
+    <!--     <box size="0.1025 0.02 0.02"/> -->
+    <!--   </geometry> -->
+    <!--   <origin xyz="-0.0707756 0 0" rpy="0 0 0"/> -->
+    <!-- </collision> -->
+    <collision>
+      <geometry>
+        <box size="0.1 0.1 0.2"/>
       </geometry>
       <origin xyz="-0.0710256 0 -0.039" rpy="0 0 0"/>
@@ -314,46 +312,46 @@
       <origin xyz="0.0 0.0 0.0" rpy="0.0 -0.0 0.0"/>
     </visual>
-    <collision>
-      <geometry>
-        <box size="0.133 0.010 0.030"/>
-      </geometry>
-      <origin xyz="-0.0459637 0.0796462 0" rpy="0 0 -1.0472"/>
-    </collision>
-    <collision>
-      <geometry>
-        <box size="0.133 0.010 0.030"/>
-      </geometry>
-      <origin xyz="-0.0459637 -0.0796462 0" rpy="0 0 1.0472"/>
-    </collision>
-    <collision>
-      <geometry>
-        <box size="0.166 0.010 0.030"/>
-      </geometry>
-      <origin xyz="-0.1699837 0.142 0" rpy="0 0 0"/>
-    </collision>
-    <collision>
-      <geometry>
-        <box size="0.166 0.010 0.030"/>
-      </geometry>
-      <origin xyz="-0.1699837 -0.142 0" rpy="0 0 0"/>
-    </collision>
-    <collision>
-      <geometry>
-        <box size="0.133 0.010 0.030"/>
-      </geometry>
-      <origin xyz="-0.2939837 0.0796462 0" rpy="0 0 1.0472"/>
-    </collision>
-    <collision>
-      <geometry>
-        <box size="0.133 0.010 0.030"/>
-      </geometry>
-      <origin xyz="-0.2939837 -0.0796462 0" rpy="0 0 -1.0472"/>
-    </collision>
-    <collision>
-      <geometry>
-        <box size="0.0465 0.034 0.0285"/>
-      </geometry>
-      <origin xyz="-0.1579837 0.166 0" rpy="0 0 0"/>
-    </collision>
+    <!-- <collision> -->
+    <!--   <geometry> -->
+    <!--     <box size="0.133 0.010 0.030"/> -->
+    <!--   </geometry> -->
+    <!--   <origin xyz="-0.0459637 0.0796462 0" rpy="0 0 -1.0472"/> -->
+    <!-- </collision> -->
+    <!-- <collision> -->
+    <!--   <geometry> -->
+    <!--     <box size="0.133 0.010 0.030"/> -->
+    <!--   </geometry> -->
+    <!--   <origin xyz="-0.0459637 -0.0796462 0" rpy="0 0 1.0472"/> -->
+    <!-- </collision> -->
+    <!-- <collision> -->
+    <!--   <geometry> -->
+    <!--     <box size="0.166 0.010 0.030"/> -->
+    <!--   </geometry> -->
+    <!--   <origin xyz="-0.1699837 0.142 0" rpy="0 0 0"/> -->
+    <!-- </collision> -->
+    <!-- <collision> -->
+    <!--   <geometry> -->
+    <!--     <box size="0.166 0.010 0.030"/> -->
+    <!--   </geometry> -->
+    <!--   <origin xyz="-0.1699837 -0.142 0" rpy="0 0 0"/> -->
+    <!-- </collision> -->
+    <!-- <collision> -->
+    <!--   <geometry> -->
+    <!--     <box size="0.133 0.010 0.030"/> -->
+    <!--   </geometry> -->
+    <!--   <origin xyz="-0.2939837 0.0796462 0" rpy="0 0 1.0472"/> -->
+    <!-- </collision> -->
+    <!-- <collision> -->
+    <!--   <geometry> -->
+    <!--     <box size="0.133 0.010 0.030"/> -->
+    <!--   </geometry> -->
+    <!--   <origin xyz="-0.2939837 -0.0796462 0" rpy="0 0 -1.0472"/> -->
+    <!-- </collision> -->
+    <!-- <collision> -->
+    <!--   <geometry> -->
+    <!--     <box size="0.0465 0.034 0.0285"/> -->
+    <!--   </geometry> -->
+    <!--   <origin xyz="-0.1579837 0.166 0" rpy="0 0 0"/> -->
+    <!-- </collision> -->
   </link>
   <link name="duct3_link">
@@ -404,14 +402,14 @@
     <collision>
       <geometry>
-        <box size="0.108 0.020 0.020"/>
-      </geometry>
-      <origin xyz="-0.0340163 0 0" rpy="0 0 0"/>
-    </collision>
-    <collision>
-      <geometry>
-        <box size="0.034 0.0285 0.0465"/>
-      </geometry>
-      <origin xyz="-0.0310163 0 -39" rpy="0 0 0"/>
-    </collision>
+        <box size="0.1 0.1 0.2"/>
+      </geometry>
+      <origin xyz="-0.0340163 0 -0.039" rpy="0 0 0"/>
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
Commit message: [hydragon] temporaly increase joint torque

File: robots/hydragon/urdf/common.xacro (robot description, xacro)
@@ -565,5 +565,5 @@
   </link>
   <joint name="front1_roll" type="revolute">
-    <limit effort="3" lower="-3.14" upper="3.14" velocity="12.5"/>
+    <limit effort="30" lower="-3.14" upper="3.14" velocity="12.5"/>
     <parent link="front1_link"/>
     <child link="body1_link"/>
@@ -572,5 +572,5 @@
   </joint>
   <joint name="gimbal1_pitch" type="revolute">
-    <limit effort="3" lower="-3.14" upper="3.14" velocity="12.5"/>
+    <limit effort="30" lower="-3.14" upper="3.14" velocity="12.5"/>
     <parent link="body1_link"/>
     <child link="duct1_link"/>
@@ -586,5 +586,5 @@
   </joint>
   <joint name="end1_roll" type="revolute">
-    <limit effort="3" lower="-3.14" upper="3.14" velocity="12.5"/>
+    <limit effort="30" lower="-3.14" upper="3.14" velocity="12.5"/>
     <parent link="body1_link"/>
     <child link="end1_link"/>
@@ -600,5 +600,5 @@
   </joint>
   <joint name="front2_roll" type="revolute">
-    <limit effort="3" lower="-3.14" upper="3.14" velocity="12.5"/>
+    <limit effort="30" lower="-3.14" upper="3.14" velocity="12.5"/>
     <parent link="front2_link"/>
     <child link="body2_link"/>
@@ -621,5 +621,5 @@
   </joint>
   <joint name="end2_roll" type="revolute">
-    <limit effort="3" lower="-3.14" upper="3.14" velocity="12.5"/>
+    <limit effort="30" lower="-3.14" upper="3.14" velocity="12.5"/>
     <parent link="body2_link"/>
     <child link="end2_link"/>
@@ -635,5 +635,5 @@
   </joint>
   <joint name="front3_roll" type="revolute">
-    <limit effort="3" lower="-3.14" upper="3.14" velocity="12.5"/>
+    <limit effort="30" lower="-3.14" upper="3.14" velocity="12.5"/>
     <parent link="front3_link"/>
     <child link="body3_link"/>
@@ -656,5 +656,5 @@
   </joint>
   <joint name="end3_roll" type="revolute">
-    <limit effort="3" lower="-3.14" upper="3.14" velocity="12.5"/>
+    <limit effort="30" lower="-3.14" upper="3.14" velocity="12.5"/>
     <parent link="body3_link"/>
     <child link="end3_link"/>
@@ -670,5 +670,5 @@
   </joint>
   <joint name="front4_roll" type="revolute">
-    <limit effort="3" lower="-3.14" upper="3.14" velocity="12.5"/>
+    <limit effort="30" lower="-3.14" upper="3.14" velocity="12.5"/>
     <parent link="front4_link"/>
     <child link="body4_link"/>
@@ -691,5 +691,5 @@
   </joint>
   <joint name="end4_roll" type="revolute">
-    <limit effort="3" lower="-3.14" upper="3.14" velocity="12.5"/>
+    <limit effort="30" lower="-3.14" upper="3.14" velocity="12.5"/>
     <parent link="body4_link"/>
     <child link="end4_link"/>
