Commit message: fix uuv_d robot parameters

File: robots/uuv_d/robots/prototype_202605/robot.gazebo.xacro (robot description, xacro)
@@ -16,13 +16,4 @@
     </gazebo>
   </xacro:macro>
-  <!-- Gazebo does not pick up the RViz-side material overrides for these meshes. -->
-  <xacro:gazebo_link_color link="t1" rgba="0.75 1.0 0.2 1.0" emissive="0.18 0.24 0.05 1.0"/>
-  <xacro:gazebo_link_color link="t2" rgba="0.75 1.0 0.2 1.0" emissive="0.18 0.24 0.05 1.0"/>
-  <xacro:gazebo_link_color link="t3" rgba="0.75 1.0 0.2 1.0" emissive="0.18 0.24 0.05 1.0"/>
-  <xacro:gazebo_link_color link="t4" rgba="0.75 1.0 0.2 1.0" emissive="0.18 0.24 0.05 1.0"/>
-  <xacro:gazebo_link_color link="t5" rgba="0.75 1.0 0.2 1.0" emissive="0.18 0.24 0.05 1.0"/>
-  <xacro:gazebo_link_color link="t6" rgba="0.75 1.0 0.2 1.0" emissive="0.18 0.24 0.05 1.0"/>
-  <xacro:gazebo_link_color link="t7" rgba="0.75 1.0 0.2 1.0" emissive="0.18 0.24 0.05 1.0"/>
-  <xacro:gazebo_link_color link="t8" rgba="0.75 1.0 0.2 1.0" emissive="0.18 0.24 0.05 1.0"/>
   <gazebo reference="root_joint">
     <disableFixedJointLumping>true</disableFixedJointLumping>
@@ -36,5 +27,5 @@
         <neutrally_buoyant>0</neutrally_buoyant>
         <!-- todo: adjust the volume according to the real robot -->
-        <volume>0.0037</volume>
+        <volume>0.0047</volume>
         <scaling_volume>1.0</scaling_volume>
         <box>
@@ -43,5 +34,5 @@
           <height>0.072</height>
         </box>
-        <center_of_buoyancy>0.000610809453814865 0 -0.1655</center_of_buoyancy>
+        <center_of_buoyancy>5.0128636417574e-06 -0.0 -0.02</center_of_buoyancy>
         <hydrodynamic_model>
           <type>fossen</type>

File: robots/uuv_d/robots/prototype_202605/robot.urdf.xacro (robot description, xacro)
@@ -3,5 +3,19 @@
   <baselink name="fc" />
   <thrust_link name="thrust" />
-  <m_f_rate value="-0.00096" />
+  <m_f_rate value="-0.02" />
+  <xacro:property name="max_force" value="20.0" />
+  <xacro:property name="min_force" value="-20.0" />
+  <xacro:macro name="thrust_link" params="name">
+    <link name="${name}">
+      <inertial>
+        <origin xyz="0 0 0" rpy="0 0 0"/>
+        <mass value="0.0091"/>
+        <inertia
+            ixx="0.00000807" ixy="0.0" ixz="0.0"
+            iyy="0.00000807" iyz="0.0"
+            izz="0.00001612"/>
+      </inertial>
+    </link>
+  </xacro:macro>
   <link name="root">
     <inertial>
@@ -22,16 +36,11 @@
     <link name="base_link">
     <inertial>
-      <origin xyz="0.000610809453814865 0 -0.165570321518981" rpy="0.0 -0.0 0.0"/>
-<mass value="2.8"/>
-<inertia ixx="0.013466428496435968"
-         ixy="7.117725680010082e-05"
-         ixz="-8.018855679667977e-11"
-         iyy="0.014514358837516688"
-         iyz="-3.042990050973674e-11"
-         izz="0.007251440331225416"/>
+      <origin xyz="5.0128636417574e-06 -0.0 -0.01" rpy="0.0 -0.0 0.0"/>
+      <mass value="4.133"/>
+      <inertia ixx="0.0222240677656555" ixy="10.28612545459733e-06" ixz="-4.8107950986871e-09" iyy="0.01243442433014907" iyz="2.67294728800918e-11" izz="0.0125174721752126"/>
     </inertial>
     <visual>
       <geometry>
-        <mesh filename="package://uuv_d/urdf/mesh/proto_type/meshes/base_link.dae"/>
+        <mesh filename="package://uuv_d/urdf/mesh/prototype_2/meshes/base_link.dae"/>
       </geometry>
       <material name="__unnamed_material_1"/>
@@ -40,460 +49,73 @@
     <collision>
       <geometry>
-        <mesh filename="package://uuv_d/urdf/mesh/proto_type/meshes/base_link.stl"/>
+        <mesh filename="package://uuv_d/urdf/mesh/prototype_2/meshes/base_link.stl"/>
       </geometry>
       <origin xyz="0.0 0.0 0.0" rpy="0.0 -0.0 0.0"/>
     </collision>
   </link>
-  <link name="t1">
-    <inertial>
-      <origin xyz="-0.014292 -0.0143 0.017717" rpy="0.0 -0.0 0.0"/>
-      <mass value="0.099392"/>
-      <inertia ixx="7.9154e-05" ixy="6.1395e-08" ixz="-3.7817e-06" iyy="7.9136e-05" iyz="-3.804e-06" izz="7.672e-05"/>
-    </inertial>
-    <visual>
-      <geometry>
-        <mesh filename="package://uuv_d/urdf/mesh/proto_type/meshes/t1.dae"/>
-      </geometry>
-      <material name="__unnamed_material_2"/>
-      <origin xyz="0.0 0.0 0.0" rpy="0.0 -0.0 0.0"/>
-    </visual>
-    <collision>
-      <geometry>
-        <mesh filename="package://uuv_d/urdf/mesh/proto_type/meshes/t1.stl"/>
-      </geometry>
-      <origin xyz="0.0 0.0 0.0" rpy="0.0 -0.0 0.0"/>
-    </collision>
-  </link>
-  <link name="thrust1">
-    <inertial>
-      <origin xyz="-1.19904086659517e-14 -2.5729418595688e-14 -0.000999999999986234" rpy="0.0 -0.0 0.0"/>
-      <mass value="0.00283424938765199"/>
-      <inertia ixx="6.52506444943004e-07" ixy="-1.05879118406788e-21" ixz="3.04402465419514e-22" iyy="6.52506444942997e-07" iyz="-3.97046694025453e-22" izz="1.30312339029423e-06"/>
-    </inertial>
-    <visual>
-      <geometry>
-        <mesh filename="package://uuv_d/urdf/mesh/proto_type/meshes/thrust1.dae"/>
-      </geometry>
-      <material name="__unnamed_material_3"/>
-      <origin xyz="0.0 0.0 0.0" rpy="0.0 -0.0 0.0"/>
-    </visual>
-    <collision>
-      <geometry>
-        <mesh filename="package://uuv_d/urdf/mesh/proto_type/meshes/thrust1.stl"/>
-      </geometry>
-      <origin xyz="0.0 0.0 0.0" rpy="0.0 -0.0 0.0"/>
-    </collision>
-  </link>
-  <link name="t2">
-    <inertial>
-      <origin xyz="-0.0143 0.014292 0.017717" rpy="0.0 -0.0 0.0"/>
-      <mass value="0.099392"/>
-      <inertia ixx="7.9136e-05" ixy="-6.1395e-08" ixz="-3.804e-06" iyy="7.9154e-05" iyz="3.7817e-06" izz="7.672e-05"/>
-    </inertial>
-    <visual>
-      <geometry>
-        <mesh filename="package://uuv_d/urdf/mesh/proto_type/meshes/t2.dae"/>
-      </geometry>
-      <material name="__unnamed_material_4"/>
-      <origin xyz="0.0 0.0 0.0" rpy="0.0 -0.0 0.0"/>
-    </visual>
-    <collision>
-      <geometry>
-        <mesh filename="package://uuv_d/urdf/mesh/proto_type/meshes/t2.stl"/>
-      </geometry>
-      <origin xyz="0.0 0.0 0.0" rpy="0.0 -0.0 0.0"/>
-    </collision>
-  </link>
-  <link name="thrust2">
-    <inertial>
-      <origin xyz="1.13242748511766e-14 2.95874436062604e-14 0.00100000000002698" rpy="0.0 -0.0 0.0"/>
-      <mass value="0.00283424938765202"/>
-      <inertia ixx="6.52506444943003e-07" ixy="5.05572790392411e-21" ixz="5.69100261436483e-22" iyy="6.52506444943006e-07" iyz="-1.05879118406788e-22" izz="1.30312339029424e-06"/>
-    </inertial>
-    <visual>
-      <geometry>
-        <mesh filename="package://uuv_d/urdf/mesh/proto_type/meshes/thrust2.dae"/>
-      </geometry>
-      <material name="__unnamed_material_5"/>
-      <origin xyz="0.0 0.0 0.0" rpy="0.0 -0.0 0.0"/>
-    </visual>
-    <collision>
-      <geometry>
-        <mesh filename="package://uuv_d/urdf/mesh/proto_type/meshes/thrust2.stl"/>
-      </geometry>
-      <origin xyz="0.0 0.0 0.0" rpy="0.0 -0.0 0.0"/>
-    </collision>
-  </link>
-  <link name="t3">
-    <inertial>
-      <origin xyz="0.014292 0.0143 0.017717" rpy="0.0 -0.0 0.0"/>
-      <mass value="0.099392"/>
-      <inertia ixx="7.9154e-05" ixy="6.1395e-08" ixz="3.7817e-06" iyy="7.9136e-05" iyz="3.804e-06" izz="7.672e-05"/>
-    </inertial>
-    <visual>
-      <geometry>
-        <mesh filename="package://uuv_d/urdf/mesh/proto_type/meshes/t3.dae"/>
-      </geometry>
-      <material name="__unnamed_material_6"/>
-      <origin xyz="0.0 0.0 0.0" rpy="0.0 -0.0 0.0"/>
-    </visual>
-    <collision>
-      <geometry>
-        <mesh filename="package://uuv_d/urdf/mesh/proto_type/meshes/t3.stl"/>
-      </geometry>
-      <origin xyz="0.0 0.0 0.0" rpy="0.0 -0.0 0.0"/>
-    </collision>
-  </link>
-  <link name="thrust3">
-    <inertial>
-      <origin xyz="-1.62092561595273e-14 2.35644836976689e-14 0.00100000000001926" rpy="0.0 -0.0 0.0"/>
-      <mass value="0.002834249387652"/>
-      <inertia ixx="6.52506444942998e-07" ixy="4.18222517706811e-21" ixz="-6.61744490042422e-23" iyy="6.52506444943007e-07" iyz="-5.29395592033938e-23" izz="1.30312339029424e-06"/>
-    </inertial>
-    <visual>
-      <geometry>
-        <mesh filename="package://uuv_d/urdf/mesh/proto_type/meshes/thrust3.dae"/>
-      </geometry>
-      <material name="__unnamed_material_7"/>
-      <origin xyz="0.0 0.0 0.0" rpy="0.0 -0.0 0.0"/>
-    </visual>
-    <collision>
-      <geometry>
-        <mesh filename="package://uuv_d/urdf/mesh/proto_type/meshes/thrust3.stl"/>
-      </geometry>
-      <origin xyz="0.0 0.0 0.0" rpy="0.0 -0.0 0.0"/>
-    </collision>
-  </link>
-  <link name="t4">
-    <inertial>
-      <origin xyz="0.0143 -0.014292 0.017717" rpy="0.0 -0.0 0.0"/>
-      <mass value="0.099392"/>
-      <inertia ixx="7.9136e-05" ixy="-6.1395e-08" ixz="3.804e-06" iyy="7.9154e-05" iyz="-3.7817e-06" izz="7.672e-05"/>
-    </inertial>
-    <visual>
-      <geometry>
-        <mesh filename="package://uuv_d/urdf/mesh/proto_type/meshes/t4.dae"/>
-      </geometry>
-      <material name="__unnamed_material_8"/>
-      <origin xyz="0.0 0.0 0.0" rpy="0.0 -0.0 0.0"/>
-    </visual>
-    <collision>
-      <geometry>
-        <mesh filename="package://uuv_d/urdf/mesh/proto_type/meshes/t4.stl"/>
-      </geometry>
-      <origin xyz="0.0 0.0 0.0" rpy="0.0 -0.0 0.0"/>
-    </collision>
-  </link>
-  <link name="thrust4">
-    <inertial>
-      <origin xyz="2.66453525910038e-15 2.57155408078802e-14 0.000999999999986345" rpy="0.0 -0.0 0.0"/>
-      <mass value="0.00283424938765204"/>
-      <inertia ixx="6.52506444943016e-07" ixy="-6.89537758624204e-21" ixz="-1.05879118406788e-22" iyy="6.52506444943005e-07" iyz="1.05879118406788e-22" izz="1.30312339029425e-06"/>
-    </inertial>
-    <visual>
-      <geometry>
-        <mesh filename="package://uuv_d/urdf/mesh/proto_type/meshes/thrust4.dae"/>
-      </geometry>
-      <material name="__unnamed_material_9"/>
-      <origin xyz="0.0 0.0 0.0" rpy="0.0 -0.0 0.0"/>
-    </visual>
-    <collision>
-      <geometry>
-        <mesh filename="package://uuv_d/urdf/mesh/proto_type/meshes/thrust4.stl"/>
-      </geometry>
-      <origin xyz="0.0 0.0 0.0" rpy="0.0 -0.0 0.0"/>
-    </collision>
-  </link>
-  <link name="t5">
-    <inertial>
-      <origin xyz="0.014292 -0.0143 -0.017717" rpy="0.0 -0.0 0.0"/>
-      <mass value="0.099392"/>
-      <inertia ixx="7.9154e-05" ixy="-6.1395e-08" ixz="-3.7817e-06" iyy="7.9136e-05" iyz="3.804e-06" izz="7.672e-05"/>
-    </inertial>
-    <visual>
-      <geometry>
-        <mesh filename="package://uuv_d/urdf/mesh/proto_type/meshes/t5.dae"/>
-      </geometry>
-      <material name="__unnamed_material_10"/>
-      <origin xyz="0.0 0.0 0.0" rpy="0.0 -0.0 0.0"/>
-    </visual>
-    <collision>
-      <geometry>
-        <mesh filename="package://uuv_d/urdf/mesh/proto_type/meshes/t5.stl"/>
-      </geometry>
-      <origin xyz="0.0 0.0 0.0" rpy="0.0 -0.0 0.0"/>
-    </collision>
-  </link>
-  <link name="thrust5">
-    <inertial>
-      <origin xyz="-3.99680288865056e-15 -8.46545056276682e-16 0.000999999999998336" rpy="0.0 -0.0 0.0"/>
-      <mass value="0.002834249387652"/>
-      <inertia ixx="6.52506444943002e-07" ixy="-7.00125670464883e-21" ixz="-1.85288457211878e-22" iyy="6.52506444943005e-07" iyz="-1.58818677610181e-22" izz="1.30312339029424e-06"/>
-    </inertial>
-    <visual>
-      <geometry>
-        <mesh filename="package://uuv_d/urdf/mesh/proto_type/meshes/thrust5.dae"/>
-      </geometry>
-      <material name="__unnamed_material_11"/>
-      <origin xyz="0.0 0.0 0.0" rpy="0.0 -0.0 0.0"/>
-    </visual>
-    <collision>
-      <geometry>
-        <mesh filename="package://uuv_d/urdf/mesh/proto_type/meshes/thrust5.stl"/>
-      </geometry>
-      <origin xyz="0.0 0.0 0.0" rpy="0.0 -0.0 0.0"/>
-    </collision>
-  </link>
-  <link name="t6">
-    <inertial>
-      <origin xyz="0.0143 0.014292 -0.017717" rpy="0.0 -0.0 0.0"/>
-      <mass value="0.099392"/>
-      <inertia ixx="7.9136e-05" ixy="6.1395e-08" ixz="-3.804e-06" iyy="7.9154e-05" iyz="-3.7817e-06" izz="7.672e-05"/>
-    </inertial>
-    <visual>
-      <geometry>
-        <mesh filename="package://uuv_d/urdf/mesh/proto_type/meshes/t6.dae"/>
-      </geometry>
-      <material name="__unnamed_material_12"/>
-      <origin xyz="0.0 0.0 0.0" rpy="0.0 -0.0 0.0"/>
-    </visual>
-    <collision>
-      <geometry>
-        <mesh filename="package://uuv_d/urdf/mesh/proto_type/meshes/t6.stl"/>
-      </geometry>
-      <origin xyz="0.0 0.0 0.0" rpy="0.0 -0.0 0.0"/>
-    </collision>
-  </link>
-  <link name="thrust6">
-    <inertial>
-      <origin xyz="-1.99840144432528e-15 1.31838984174237e-15 0.00099999999999012" rpy="0.0 -0.0 0.0"/>
-      <mass value="0.00283424938765201"/>
-      <inertia ixx="6.52506444943003e-07" ixy="-5.9557004103818e-22" ixz="-1.98523347012727e-22" iyy="6.52506444942998e-07" iyz="1.05879118406788e-22" izz="1.30312339029423e-06"/>
-    </inertial>
-    <visual>
-      <geometry>
-        <mesh filename="package://uuv_d/urdf/mesh/proto_type/meshes/thrust6.dae"/>
-      </geometry>
-      <material name="__unnamed_material_13"/>
-      <origin xyz="0.0 0.0 0.0" rpy="0.0 -0.0 0.0"/>
-    </visual>
-    <collision>
-      <geometry>
-        <mesh filename="package://uuv_d/urdf/mesh/proto_type/meshes/thrust6.stl"/>
-      </geometry>
-      <origin xyz="0.0 0.0 0.0" rpy="0.0 -0.0 0.0"/>
-    </collision>
-  </link>
-  <link name="t7">
-    <inertial>
-      <origin xyz="-0.014292 0.0143 -0.017717" rpy="0.0 -0.0 0.0"/>
-      <mass value="0.099392"/>
-      <inertia ixx="7.9154e-05" ixy="-6.1395e-08" ixz="3.7817e-06" iyy="7.9136e-05" iyz="-3.804e-06" izz="7.672e-05"/>
-    </inertial>
-    <visual>
-      <geometry>
-        <mesh filename="package://uuv_d/urdf/mesh/proto_type/meshes/t7.dae"/>
-      </geometry>
-      <material name="__unnamed_material_14"/>
-      <origin xyz="0.0 0.0 0.0" rpy="0.0 -0.0 0.0"/>
-    </visual>
-    <collision>
-      <geometry>
-        <mesh filename="package://uuv_d/urdf/mesh/proto_type/meshes/t7.stl"/>
-      </geometry>
-      <origin xyz="0.0 0.0 0.0" rpy="0.0 -0.0 0.0"/>
-    </collision>
-  </link>
-  <link name="thrust7">
-    <inertial>
-      <origin xyz="1.4210854715202e-14 -1.01862962509358e-14 0.00100000000002154" rpy="0.0 -0.0 0.0"/>
-      <mass value="0.002834249387652"/>
-      <inertia ixx="6.52506444943e-07" ixy="-7.05419626385222e-21" ixz="-1.31157757926408e-20" iyy="6.52506444942999e-07" iyz="1.03496838242635e-20" izz="1.30312339029423e-06"/>
-    </inertial>
-    <visual>
-      <geometry>
-        <mesh filename="package://uuv_d/urdf/mesh/proto_type/meshes/thrust7.dae"/>
-      </geometry>
-      <material name="__unnamed_material_15"/>
-      <origin xyz="0.0 0.0 0.0" rpy="0.0 -0.0 0.0"/>
-    </visual>
-    <collision>
-      <geometry>
-        <mesh filename="package://uuv_d/urdf/mesh/proto_type/meshes/thrust7.stl"/>
-      </geometry>
-      <origin xyz="0.0 0.0 0.0" rpy="0.0 -0.0 0.0"/>
-    </collision>
-  </link>
-  <link name="t8">
-    <inertial>
-      <origin xyz="-0.0143 -0.014292 -0.017717" rpy="0.0 -0.0 0.0"/>
-      <mass value="0.099392"/>
-      <inertia ixx="7.9136e-05" ixy="6.1395e-08" ixz="3.804e-06" iyy="7.9154e-05" iyz="3.7817e-06" izz="7.672e-05"/>
-    </inertial>
-    <visual>
-      <geometry>
-        <mesh filename="package://uuv_d/urdf/mesh/proto_type/meshes/t8.dae"/>
-      </geometry>
-      <material name="__unnamed_material_16"/>
-      <origin xyz="0.0 0.0 0.0" rpy="0.0 -0.0 0.0"/>
-    </visual>
-    <collision>
-      <geometry>
-        <mesh filename="package://uuv_d/urdf/mesh/proto_type/meshes/t8.stl"/>
-      </geometry>
-      <origin xyz="0.0 0.0 0.0" rpy="0.0 -0.0 0.0"/>
-    </collision>
-  </link>
-  <link name="thrust8">
-    <inertial>
-      <origin xyz="-4.66293670342566e-15 3.76088049591772e-15 0.00100000000000233" rpy="0.0 -0.0 0.0"/>
-      <mass value="0.00283424938765202"/>
-      <inertia ixx="6.52506444942999e-07" ixy="-6.04834463898774e-21" ixz="-1.45583787809333e-22" iyy="6.52506444943014e-07" iyz="-2.38228016415272e-22" izz="1.30312339029425e-06"/>
-    </inertial>
-    <visual>
-      <geometry>
-        <mesh filename="package://uuv_d/urdf/mesh/proto_type/meshes/thrust8.dae"/>
-      </geometry>
-      <material name="__unnamed_material_17"/>
-      <origin xyz="0.0 0.0 0.0" rpy="0.0 -0.0 0.0"/>
-    </visual>
-    <collision>
-      <geometry>
-        <mesh filename="package://uuv_d/urdf/mesh/proto_type/meshes/thrust8.stl"/>
-      </geometry>
-      <origin xyz="0.0 0.0 0.0" rpy="0.0 -0.0 0.0"/>
-    </collision>
-  </link>
-  <link name="fc">
-    <inertial>
-      <origin xyz="0.0 0.0 0.0" rpy="0.0 -0.0 0.0"/>
-      <mass value="0.0"/>
-      <inertia ixx="0.0" ixy="0.0" ixz="0.0" iyy="0.0" iyz="0.0" izz="0.0"/>
-    </inertial>
-    <visual>
-      <geometry>
-        <mesh filename="package://uuv_d/urdf/mesh/proto_type/meshes/fc.dae"/>
-      </geometry>
-      <material name="__unnamed_material_18"/>
-      <origin xyz="0.0 0.0 0.0" rpy="0.0 -0.0 0.0"/>
-    </visual>
-    <collision>
-      <geometry>
-        <mesh filename="package://uuv_d/urdf/mesh/proto_type/meshes/fc.stl"/>
-      </geometry>
-      <origin xyz="0.0 0.0 0.0" rpy="0.0 -0.0 0.0"/>
-    </collision>
-  </link>
-  <joint name="l1" type="fixed">
-    <limit effort="0.0" velocity="0.0" lower="-20.0" upper="20.0"/>
-    <parent link="base_link"/>
-    <child link="t1"/>
-    <axis xyz="0. 0. 0."/>
-    <origin xyz="0.109644792463034 0.0969168704014227 -0.281585755800395" rpy="0.0 -0.0 0.0"/>
-  </joint>
+  <xacro:thrust_link name="thrust1"/>
+  <xacro:thrust_link name="thrust2"/>
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